File: EAGLE CAD/Modular_RFPA_v105.brd (EAGLE design)
At the start: 152.4 x 152.4 mm, 197 parts, among them IC201 74AHC1G14DBV, IC202 LM324D, J1 FUSE_2P, J2 KK_PCFAN, Q1 IRF540, Q101 IRF540, Q102 IRF540, Q2 IRF540, Q201 BSS123, T1 HP4_TRAFO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

Commit message: Work on IRF630 PA
Also add FET_parameters_sheet.csv
add IRF520 and IRF520N datasheets
Parts:
- C102, C104: value 0.1uF -> 22nF
- C105: value 0.1uF -> 12nF
- C106, C107, C109, C110, C17, C24, C25, C26, C27: value 0.1uF -> DNP
- C111, C112: value 22nF -> 2.2nF
- C113, C114: value 0.1uF -> 10nF
- C29: value 0.1uF -> SHORT
- L101, L102: value 1uH -> 150nH
- L6: value DR127 -> 22uH
- Q101: value IRF540 -> IRF630
- Q102: value IRF540 -> IRF520N
- R101, R105: value 1K -> 75
- R102, R106: value 1K -> 150
- R103: value 1K -> 4.99
- R104: value 1K -> 10
- R107, R109: value 1.0K -> 100
- R108, R110: value 1K -> 100
- R111, R112, R115, R116: value 1.0K -> DNP
- R113, R114: value 1.0K -> 15
- R117: value 1K -> 330
- R118, R120: value 1K -> 270
- R119: value 1K -> 2.74K
- R121, R123, R34: value 1K -> 2.7
- R122, R124: value 1K -> 6.8
- R30: value 1.0K -> 0
- R32, R33: value 1K -> 8.2
- R35: value 1K -> 3.3
- R40: value 0.33 -> 1.0
- R43: value 0.33 -> 0.5

Commit message: Change Ldamp from 150nH to 47nH
Parts:
- L101: value 150nH -> 47nH
Changed lines of the file:
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@@
 <attribute name="POWER" value="0.25" x="74.676" y="97.79" size="1.778" layer="27" rot="R270" display="off"/>
 </element>
-<element name="L101" library="MDT_L" package="L1008" value="150nH" x="67.564" y="92.71" rot="R180">
+<element name="L101" library="MDT_L" package="L1008" value="47nH" x="67.564" y="92.71" rot="R180">
 <attribute name="PACKAGE" value="1008" x="67.564" y="92.71" size="1.778" layer="27" rot="R180" display="off"/>
 <attribute name="IDC" value="0.37A" x="67.564" y="92.71" size="1.778" layer="27" rot="R180" display="off"/>

Commit message: Update component values for gate bias driver
Change C209 from 220pF to 330pF
Parts:
- C103: value 0.1uF -> 27nF
- C207: value 0.1uF -> DNP
- C208: value 0.1uF -> 1nF
- C209: value 0.1uF -> 330pF
- C28: value 0.1uF -> 47nF
- C29: value SHORT -> 100nF
- R201: value (none) -> 10K
- R202, R203, R204, R205, R206, R212, R219: value 1.0K -> 10K
- R211, R214: value 1.0K -> DNP
- R216: value 1.0K -> 0
- R217: value 1.0K -> 10
- R218: value 1.0K -> 33.2
- R41: value 1.0K -> 150

Commit message: Done testing for today
Seem to be getting significant loss across baluns
Measured input balun leakage at ~650nH (primary referred, both secondaries shorted to gnd)
Parts:
- C25: value DNP -> 1.5nF
- C28: value 47nF -> DNP
Changed lines of the file:
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@@
 <attribute name="POWER" value="" x="90.17" y="27.94" size="1.778" layer="27" rot="R270" display="off"/>
 </element>
-<element name="C25" library="MDT_C" package="0805_IPC-7351B" value="DNP" x="50.8" y="10.16" rot="R270">
+<element name="C25" library="MDT_C" package="0805_IPC-7351B" value="1.5nF" x="50.8" y="10.16" rot="R270">
 <attribute name="PACKAGE" value="0805" x="50.8" y="10.16" size="1.778" layer="27" font="vector" ratio="10" rot="R270" display="off"/>
 <attribute name="PARTNO" value="" x="50.8" y="10.16" size="1.778" layer="27" font="vector" ratio="10" rot="R270" display="off"/>
@@
 <attribute name="DIALECTRIC" value="" x="46.99" y="10.16" size="1.778" layer="27" font="vector" ratio="10" rot="R270" display="off"/>
 </element>
-<element name="C28" library="MDT_C" package="0805_IPC-7351B" value="47nF" x="43.18" y="10.16" rot="R270">
+<element name="C28" library="MDT_C" package="0805_IPC-7351B" value="DNP" x="43.18" y="10.16" rot="R270">
 <attribute name="PACKAGE" value="0805" x="43.18" y="10.16" size="1.778" layer="27" font="vector" ratio="10" rot="R270" display="off"/>
 <attribute name="PARTNO" value="" x="43.18" y="10.16" size="1.778" layer="27" font="vector" ratio="10" rot="R270" display="off"/>
