File: EAGLE CAD/Modular_RFPA_v105.brd (EAGLE design)
At the start: 152.4 x 152.4 mm, 197 parts, among them IC201 74AHC1G14DBV, IC202 LM324D, J1 FUSE_2P, J2 KK_PCFAN, Q1 IRF540, Q101 IRF630, Q102 IRF520N, Q2 IRF540, Q201 BSS123, T1 HP4_TRAFO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

Commit message: more assembly variant work....
Parts:
- C15, C16: value 47nF -> 4.7uF
- R302, R303: value 1K -> 1.0
Routing:
- net +5V: track 159.8 -> 153.5 mm
- net +12V: track 143.7 -> 137.4 mm
