File: EAGLE CAD/Modular_RFPA_v105.brd (EAGLE design)
At the start: 152.4 x 152.4 mm, 197 parts, among them IC201 74AHC1G14DBV, IC202 LM324D, J1 FUSE_2P, J2 KK_PCFAN, Q1 IRF540, Q101 IRF630, Q102 IRF520N, Q2 IRF540, Q201 BSS123, T1 HP4_TRAFO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

Commit message: change a couple bias driver components
need to rework the 01 board like this too
Parts:
- C208: value 1nF -> DNP
- C209: value 330pF -> 15pF
- R218: value 33.2 -> 100
Changed lines of the file:
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@@
 </attributes>
 <variantdefs>
-<variantdef name="IRF520N_20W"/>
+<variantdef name="IRF520N_20W" current="yes"/>
 <variantdef name="IRF630_200W"/>
 </variantdefs>
@@
 <attribute name="POWER" value="1" x="65.532" y="87.63" size="1.778" layer="27" rot="R180" display="off"/>
 <variant name="IRF520N_20W" value="2.74K"/>
-<variant name="IRF630_200W" value="117"/>
 </element>
 <element name="R113" library="MDT_R" package="0805_IPC-7351B" value="15" x="67.564" y="96.266" rot="R180">
@@
 <attribute name="POWER" value="" x="116.84" y="33.274" size="1.778" layer="27" rot="R90" display="off"/>
 </element>
-<element name="R218" library="MDT_R" package="0805_IPC-7351B" value="33.2" x="116.84" y="38.608" rot="R90">
+<element name="R218" library="MDT_R" package="0805_IPC-7351B" value="100" x="116.84" y="38.608" rot="R90">
 <attribute name="PACKAGE" value="0805" x="116.84" y="38.608" size="1.778" layer="27" rot="R90" display="off"/>
 <attribute name="PARTNO" value="" x="116.84" y="38.608" size="1.778" layer="27" rot="R90" display="off"/>
@@
 <attribute name="POWER" value="" x="102.108" y="16.764" size="1.778" layer="27" rot="R180" display="off"/>
 </element>
-<element name="C209" library="MDT_C" package="0805_IPC-7351B" value="330pF" x="110.744" y="29.464" rot="R180">
+<element name="C209" library="MDT_C" package="0805_IPC-7351B" value="15pF" x="110.744" y="29.464" rot="R180">
 <attribute name="PACKAGE" value="0805" x="110.744" y="29.464" size="1.778" layer="27" rot="R180" display="off"/>
 <attribute name="PARTNO" value="" x="110.744" y="29.464" size="1.778" layer="27" rot="R180" display="off"/>
@@
 <variant name="IRF630_200W" populate="no"/>
 </element>
-<element name="C208" library="MDT_C" package="0805_IPC-7351B" value="1nF" x="101.092" y="33.02" rot="R90">
+<element name="C208" library="MDT_C" package="0805_IPC-7351B" value="DNP" x="101.092" y="33.02" rot="R90">
 <attribute name="PACKAGE" value="0805" x="101.092" y="33.02" size="1.778" layer="27" rot="R90" display="off"/>
 <attribute name="PARTNO" value="" x="101.092" y="33.02" size="1.778" layer="27" rot="R90" display="off"/>
@@
 <attribute name="TOL" value="" x="101.092" y="33.02" size="1.778" layer="27" rot="R90" display="off"/>
 <attribute name="DIALECTRIC" value="" x="101.092" y="33.02" size="1.778" layer="27" rot="R90" display="off"/>
+<variant name="IRF520N_20W" populate="no"/>
+<variant name="IRF630_200W" populate="no"/>
 </element>
 <element name="C201" library="MDT_C" package="0805_IPC-7351B" value="0.1uF" x="112.776" y="23.622" rot="R90">

Commit message: More schematic editing
Add DR127 to my library
More assembly variant component values
Parts:
- C1, C7: value 22nF -> 2.2nF
- C11, C5: value 0.1uF -> 27nF
- C12, C6: value 0.1uF -> 22nF
- C2, C8: value 0.1uF -> 10nF
- L1, L2: value 1uH -> 47nH
- L6: value 22uH -> (none); device inductors:DR127 -> MDT_L:DR127
- L7: value DR127 -> (none); device inductors:DR127 -> MDT_L:DR127
- Q1, Q2: value IRF540 -> IRF630
- R1, R14: value 1K -> 270
- R12, R25: value 1.0K -> 100
- R13, R18, R26, R5: value 1K -> 75
- R15, R16, R2, R3, R36, R38: value 1K -> 2.7
- R17, R4: value 1K -> 100
- R19, R6: value 1K -> 4.99
- R20, R7: value 1K -> 330
- R21, R8: value 1.0K -> 15
- R37, R39: value 1K -> 3.3
Routing:
- net DRAINS_POS: track 125.7 -> 117.1 mm
- net DRAINS_NEG: track 136.9 -> 128.3 mm
- net VB: track 28.3 -> 23.0 mm

Commit message: Work on libraries...
Parts:
- C1, C111, C112, C7: value 2.2nF -> 22nF
- C102, C104, C12, C6: value 22nF -> 0.1uF
- C103, C11, C5: value 27nF -> 0.1uF
- C105: value 12nF -> 0.1uF
- C106, C107, C109, C110, C17, C207, C208, C24, C26, C27, C28: value DNP -> 0.1uF
- C113, C114, C2, C8: value 10nF -> 0.1uF
- C15, C16: value 4.7uF -> 47nF
- C209: value 15pF -> 0.1uF
- C25: value 1.5nF -> 0.1uF
- C29: value 100nF -> 0.1uF
- L1, L101, L2: value 47nH -> 1uH
- L102: value 150nH -> 1uH
- L4, L5: device inductors:DR127 -> MDT_L:DR127
- R1, R118, R120, R14: value 270 -> 1K
- R101, R105, R13, R18, R26, R5: value 75 -> 1K
- R102, R106: value 150 -> 1K
- R103, R19, R6: value 4.99 -> 1K
- R104: value 10 -> 1K
- R107, R109, R12, R218, R25: value 100 -> 1.0K
- R108, R110, R17, R4: value 100 -> 1K
- R111, R112, R115, R116, R211, R214: value DNP -> 1.0K
- R113, R114, R21, R8: value 15 -> 1.0K
- R117, R20, R7: value 330 -> 1K
- R119: value 2.74K -> 1K
- R121, R123, R15, R16, R2, R3, R34, R36, R38: value 2.7 -> 1K
- R122, R124: value 6.8 -> 1K
- R202, R203, R204, R205, R206, R212, R219: value 10K -> 1.0K
- R216, R30: value 0 -> 1.0K
- R217: value 10 -> 1.0K
- R302, R303, R40: value 1.0 -> 1K
- R32, R33: value 8.2 -> 1K
- R35, R37, R39: value 3.3 -> 1K
- R41: value 150 -> 1.0K
- R43: value 0.5 -> 1K
