File: EAGLE CAD/Modular_RFPA_v105.sch (EAGLE design)
At the start: 197 parts, among them IC201 74AHC1G14DBV, IC202 LM324D, J1 FUSE_2P, J2 KK_PCFAN, Q1 IRF540, Q101 IRF630, Q102 IRF520N, Q2 IRF540, Q201 BSS123, T1 HP4_TRAFO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

Commit message: more assembly variant work....
Parts:
- C15, C16: value 47nF -> 4.7uF
- R302, R303: value 1K -> 1.0
Other:
- moved on the sheet: C1, C10, C11, C12, C2, C3, C4, C5, C6, C7, C8, C9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
