File: EAGLE CAD/DICO_v100.sch (EAGLE design)
At the start: 30 parts, among them T1 TRAFO_CURRENTSENSEPA1005.020Q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, T2 TRAFO_CURRENTSENSEPA1005.020Q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

Commit message: working on dico again
Connections:
- net GND: now also T1.SS, T2.SS; no longer T1.SF, T2.SF
- net N$1: now also T1.SF, T2.PS; no longer T1.SS, T2.PF
- net N$11: now also J2.1
- net N$2: now also T1.PS, T2.SF; no longer T1.PF, T2.SS
- net N$3: now also T1.PF; no longer T1.PS
- net N$8: now also T2.PF; no longer T2.PS
Changed lines of the file:
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@@
 </plain>
 <instances>
-<instance part="T1" gate="G$1" x="53.34" y="53.34" rot="MR0"/>
-<instance part="T2" gate="G$1" x="53.34" y="27.94" rot="MR180"/>
+<instance part="T1" gate="G$1" x="53.34" y="53.34"/>
+<instance part="T2" gate="G$1" x="53.34" y="27.94" rot="R180"/>
 <instance part="SUPPLY1" gate="GND" x="38.1" y="35.56" smashed="yes"/>
 <instance part="R1" gate="G$1" x="104.14" y="17.78"/>
@@
 <net name="N$1" class="0">
 <segment>
-<pinref part="T2" gate="G$1" pin="PF"/>
-<wire x1="66.04" y1="25.4" x2="83.82" y2="25.4" width="0.1524" layer="91"/>
 <wire x1="83.82" y1="25.4" x2="83.82" y2="50.8" width="0.1524" layer="91"/>
-<pinref part="T1" gate="G$1" pin="SS"/>
-<wire x1="83.82" y1="50.8" x2="66.04" y2="50.8" width="0.1524" layer="91"/>
 <wire x1="83.82" y1="25.4" x2="104.14" y2="25.4" width="0.1524" layer="91"/>
-<junction x="83.82" y="25.4"/>
 <pinref part="R1" gate="G$1" pin="1"/>
 <wire x1="104.14" y1="22.86" x2="104.14" y2="25.4" width="0.1524" layer="91"/>
@@
 <wire x1="116.84" y1="35.56" x2="116.84" y2="25.4" width="0.1524" layer="91"/>
 <junction x="116.84" y="25.4"/>
+<pinref part="T1" gate="G$1" pin="SF"/>
+<wire x1="83.82" y1="50.8" x2="66.04" y2="50.8" width="0.1524" layer="91"/>
+<pinref part="T2" gate="G$1" pin="PS"/>
+<wire x1="66.04" y1="25.4" x2="83.82" y2="25.4" width="0.1524" layer="91"/>
+<junction x="83.82" y="25.4"/>
 </segment>
 </net>
 <net name="N$2" class="0">
 <segment>
-<pinref part="T2" gate="G$1" pin="SS"/>
-<wire x1="40.64" y1="30.48" x2="27.94" y2="30.48" width="0.1524" layer="91"/>
 <wire x1="27.94" y1="30.48" x2="27.94" y2="55.88" width="0.1524" layer="91"/>
-<pinref part="T1" gate="G$1" pin="PF"/>
+<pinref part="C5" gate="G$1" pin="2"/>
+<wire x1="27.94" y1="55.88" x2="-5.08" y2="55.88" width="0.1524" layer="91"/>
+<pinref part="T1" gate="G$1" pin="PS"/>
 <wire x1="27.94" y1="55.88" x2="40.64" y2="55.88" width="0.1524" layer="91"/>
 <junction x="27.94" y="55.88"/>
-<pinref part="C5" gate="G$1" pin="2"/>
-<wire x1="27.94" y1="55.88" x2="-5.08" y2="55.88" width="0.1524" layer="91"/>
-</segment>
-</net>
-<net name="N$3" class="0">
-<segment>
-<pinref part="T1" gate="G$1" pin="PS"/>
-<wire x1="66.04" y1="55.88" x2="104.14" y2="55.88" width="0.1524" layer="91"/>
-<pinref part="C6" gate="G$1" pin="1"/>
+<pinref part="T2" gate="G$1" pin="SF"/>
+<wire x1="27.94" y1="30.48" x2="40.64" y2="30.48" width="0.1524" layer="91"/>
 </segment>
 </net>
 <net name="GND" class="0">
 <segment>
-<pinref part="T1" gate="G$1" pin="SF"/>
 <pinref part="SUPPLY1" gate="GND" pin="GND"/>
-<wire x1="40.64" y1="50.8" x2="38.1" y2="50.8" width="0.1524" layer="91"/>
 <wire x1="38.1" y1="50.8" x2="38.1" y2="40.64" width="0.1524" layer="91"/>
-<pinref part="T2" gate="G$1" pin="SF"/>
 <wire x1="38.1" y1="40.64" x2="38.1" y2="38.1" width="0.1524" layer="91"/>
-<wire x1="66.04" y1="30.48" x2="68.58" y2="30.48" width="0.1524" layer="91"/>
 <wire x1="38.1" y1="40.64" x2="68.58" y2="40.64" width="0.1524" layer="91"/>
 <wire x1="68.58" y1="40.64" x2="68.58" y2="30.48" width="0.1524" layer="91"/>
 <junction x="38.1" y="40.64"/>
+<pinref part="T1" gate="G$1" pin="SS"/>
+<wire x1="40.64" y1="50.8" x2="38.1" y2="50.8" width="0.1524" layer="91"/>
+<pinref part="T2" gate="G$1" pin="SS"/>
+<wire x1="66.04" y1="30.48" x2="68.58" y2="30.48" width="0.1524" layer="91"/>
 </segment>
 <segment>
@@
 <wire x1="2.54" y1="35.56" x2="2.54" y2="25.4" width="0.1524" layer="91"/>
 <junction x="2.54" y="25.4"/>
-<pinref part="T2" gate="G$1" pin="PS"/>
+<pinref part="T2" gate="G$1" pin="PF"/>
 <wire x1="40.64" y1="25.4" x2="15.24" y2="25.4" width="0.1524" layer="91"/>
 <junction x="15.24" y="25.4"/>
@@
 <wire x1="-66.04" y1="20.32" x2="-66.04" y2="25.4" width="0.1524" layer="91"/>
 <junction x="-66.04" y="25.4"/>
+<pinref part="J2" gate="G$1" pin="1"/>
+<wire x1="-78.74" y1="25.4" x2="-101.6" y2="25.4" width="0.1524" layer="91"/>
+<junction x="-78.74" y="25.4"/>
 </segment>
 </net>
@@
 </segment>
 </net>
+<net name="N$3" class="0">
+<segment>
+<pinref part="T1" gate="G$1" pin="PF"/>
+<pinref part="C6" gate="G$1" pin="1"/>
+<wire x1="66.04" y1="55.88" x2="104.14" y2="55.88" width="0.1524" layer="91"/>
+</segment>
+</net>

Commit message: save eagle and commit again...
Parts:
- R10, R11: device MDT_R:RR-1.0K-1%-1206-0.25WR1206 -> MDT_R:R90R-1.0K-1%-1206-0.25WR1206
Other:
- moved on the sheet: R10, R11
Changed lines of the file:
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@@
 <layer number="106" name="BGA-Top" color="7" fill="1" visible="yes" active="yes"/>
 <layer number="107" name="BD-Top" color="7" fill="1" visible="yes" active="yes"/>
+<layer number="108" name="BOM" color="7" fill="1" visible="yes" active="yes"/>
+<layer number="109" name="VOLTAGE" color="7" fill="1" visible="yes" active="yes"/>
+<layer number="110" name="DEVICE" color="7" fill="1" visible="yes" active="yes"/>
+<layer number="111" name="PARTNO" color="7" fill="1" visible="yes" active="yes"/>
+<layer number="112" name="PACKAGE" color="7" fill="1" visible="yes" active="yes"/>
+<layer number="113" name="CURRENT" color="7" fill="1" visible="yes" active="yes"/>
+<layer number="114" name="TOL" color="7" fill="1" visible="yes" active="yes"/>
+<layer number="115" name="POWER" color="7" fill="1" visible="yes" active="yes"/>
 <layer number="151" name="HeatSink" color="7" fill="1" visible="yes" active="yes"/>
 <layer number="200" name="200bmp" color="7" fill="1" visible="yes" active="yes"/>
@@
 <part name="R8" library="MDT_R" deviceset="R" device="R1206" technology="R-1.0K-1%-1206-0.25W" value="1K"/>
 <part name="R9" library="MDT_R" deviceset="R" device="R1206" technology="R-1.0K-1%-1206-0.25W" value="1K"/>
-<part name="R10" library="MDT_R" deviceset="R" device="R1206" technology="R-1.0K-1%-1206-0.25W" value="1K"/>
-<part name="R11" library="MDT_R" deviceset="R" device="R1206" technology="R-1.0K-1%-1206-0.25W" value="1K"/>
+<part name="R10" library="MDT_R" deviceset="R90" device="R1206" technology="R-1.0K-1%-1206-0.25W" value="1K"/>
+<part name="R11" library="MDT_R" deviceset="R90" device="R1206" technology="R-1.0K-1%-1206-0.25W" value="1K"/>
 <part name="R12" library="MDT_R" deviceset="R" device="R1206" technology="R-1.0K-1%-1206-0.25W" value="1K"/>
 <part name="R13" library="MDT_R" deviceset="R" device="R1206" technology="R-1.0K-1%-1206-0.25W" value="1K"/>
@@
 <instance part="R8" gate="G$1" x="15.24" y="17.78" rot="MR0"/>
 <instance part="R9" gate="G$1" x="5.08" y="17.78" rot="MR0"/>
-<instance part="R10" gate="G$1" x="-5.08" y="25.4" smashed="yes" rot="MR90">
-<attribute name="NAME" x="-5.08" y="30.48" size="1.6764" layer="95" rot="MR0" align="bottom-center"/>
-<attribute name="VALUE" x="-5.08" y="28.575" size="1.6764" layer="96" rot="MR0" align="bottom-center"/>
-<attribute name="PACKAGE" x="-5.08" y="26.67" size="1.6764" layer="97" rot="MR0" align="bottom-center"/>
-<attribute name="BOM" x="-9.652" y="26.67" size="1.6764" layer="97" rot="MR90"/>
-</instance>
-<instance part="R11" gate="G$1" x="-5.08" y="35.56" smashed="yes" rot="MR90">
-<attribute name="NAME" x="-5.08" y="40.64" size="1.6764" layer="95" rot="MR0" align="bottom-center"/>
-<attribute name="VALUE" x="-5.08" y="38.735" size="1.6764" layer="96" rot="MR0" align="bottom-center"/>
-<attribute name="PACKAGE" x="-5.08" y="36.83" size="1.6764" layer="97" rot="MR0" align="bottom-center"/>
-<attribute name="BOM" x="-9.652" y="36.83" size="1.6764" layer="97" rot="MR90"/>
-</instance>
+<instance part="R10" gate="G$1" x="-5.08" y="25.4" rot="MR0"/>
+<instance part="R11" gate="G$1" x="-5.08" y="35.56" rot="MR0"/>
 <instance part="R12" gate="G$1" x="-15.24" y="17.78" rot="MR0"/>
 <instance part="R13" gate="G$1" x="-25.4" y="17.78" rot="MR0"/>
