File: EAGLE CAD/DICO_giangrandi_v100.brd (EAGLE design)
At the start: 76.2 x 50.8 mm, 32 parts, among them T1 TRAFO_CURRENTSENSEPA1005.020Q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, T2 TRAFO_CURRENTSENSEPA1005.020Q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

Commit message: DICO layout
Connections:
- net GND: now also T2.3; no longer T2.1
- net N$1: now also C7.2, R10.1, R11.1, R8.1, R9.1, T2.7; no longer C8.2, R1.1, R2.1, R3.1, R4.1, T2.8
- net N$2: no longer T2.3
- net N$3: now also T2.1
- net N$8: now also C8.2, R1.1, R2.1, R3.1, R4.1, T2.8; no longer C7.2, R10.1, R11.1, R8.1, R9.1, T2.7
Changed lines of the file:
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@@
 <signals>
 <signal name="N$1">
-<contactref element="R1" pad="1"/>
-<contactref element="R3" pad="1"/>
-<contactref element="R2" pad="1"/>
-<contactref element="R4" pad="1"/>
 <contactref element="T1" pad="3"/>
-<contactref element="T2" pad="8"/>
-<contactref element="C8" pad="2"/>
-<wire x1="2.6162" y1="-6.35" x2="-48.13" y2="-49.53" width="0" layer="19" extent="1-1"/>
-<wire x1="6.35" y1="-6.198" x2="2.6162" y2="-6.35" width="0" layer="19" extent="1-1"/>
-<wire x1="8.89" y1="-6.198" x2="6.35" y2="-6.198" width="0" layer="19" extent="1-1"/>
-<wire x1="8.738" y1="-3.81" x2="8.89" y2="-6.198" width="0" layer="19" extent="1-1"/>
-<wire x1="8.738" y1="-1.27" x2="8.738" y2="-3.81" width="0" layer="19" extent="1-1"/>
-<wire x1="1.8542" y1="1.651" x2="8.738" y2="-1.27" width="0" layer="19" extent="1-1"/>
+<contactref element="R8" pad="1"/>
+<contactref element="R10" pad="1"/>
+<contactref element="R9" pad="1"/>
+<contactref element="R11" pad="1"/>
+<contactref element="T2" pad="7"/>
+<contactref element="C7" pad="2"/>
+<wire x1="-8.89" y1="-7.468" x2="-48.13" y2="-43.18" width="0" layer="19" extent="1-1"/>
+<wire x1="-8.738" y1="-5.08" x2="-8.89" y2="-7.468" width="0" layer="19" extent="1-1"/>
+<wire x1="-6.35" y1="-7.468" x2="-8.89" y2="-7.468" width="0" layer="19" extent="1-1"/>
+<wire x1="-8.738" y1="-2.54" x2="-8.738" y2="-5.08" width="0" layer="19" extent="1-1"/>
+<wire x1="-2.6162" y1="-6.35" x2="-6.35" y2="-7.468" width="0" layer="19" extent="1-1"/>
+<wire x1="1.8542" y1="1.651" x2="-2.6162" y2="-6.35" width="0" layer="19" extent="1-1"/>
 </signal>
 <signal name="N$2">
 <contactref element="C5" pad="2"/>
 <contactref element="T1" pad="8"/>
-<contactref element="T2" pad="3"/>
 <contactref element="C7" pad="1"/>
-<wire x1="-1.8542" y1="-2.921" x2="-50.93" y2="-43.18" width="0" layer="19" extent="1-1"/>
-<wire x1="-2.6162" y1="5.08" x2="-1.8542" y2="-2.921" width="0" layer="19" extent="1-1"/>
-<wire x1="-6.94" y1="5.08" x2="-2.6162" y2="5.08" width="0" layer="19" extent="1-1"/>
+<wire x1="-6.94" y1="5.08" x2="-50.93" y2="-43.18" width="0" layer="19" extent="1-1"/>
+<wire x1="-2.6162" y1="5.08" x2="-6.94" y2="5.08" width="0" layer="19" extent="1-1"/>
 </signal>
 <signal name="GND">
@@
 <contactref element="R14" pad="2"/>
 <contactref element="T1" pad="1"/>
-<contactref element="T2" pad="1"/>
 <contactref element="J2" pad="G4"/>
 <contactref element="J2" pad="G1"/>
@@
 <contactref element="J1" pad="G2"/>
 <contactref element="J1" pad="G3"/>
+<contactref element="T2" pad="3"/>
 <wire x1="-26.56" y1="-22.61" x2="-27.56" y2="-22.61" width="0" layer="19" extent="1-16"/>
 <wire x1="-19.16" y1="-22.61" x2="-26.56" y2="-22.61" width="0" layer="19" extent="16-16"/>
@@
 <wire x1="-8.89" y1="-10.312" x2="-12.7" y2="-10.312" width="0" layer="19" extent="1-1"/>
 <wire x1="-6.35" y1="-10.312" x2="-8.89" y2="-10.312" width="0" layer="19" extent="1-1"/>
-<wire x1="1.8542" y1="-2.921" x2="-6.35" y2="-10.312" width="0" layer="19" extent="1-1"/>
-<wire x1="-1.8542" y1="1.651" x2="1.8542" y2="-2.921" width="0" layer="19" extent="1-1"/>
-<wire x1="6.35" y1="-9.042" x2="1.8542" y2="-2.921" width="0" layer="19" extent="1-1"/>
+<wire x1="-1.8542" y1="-2.921" x2="-6.35" y2="-10.312" width="0" layer="19" extent="1-1"/>
+<wire x1="-1.8542" y1="1.651" x2="-1.8542" y2="-2.921" width="0" layer="19" extent="1-1"/>
+<wire x1="6.35" y1="-9.042" x2="-1.8542" y2="-2.921" width="0" layer="19" extent="1-1"/>
 <wire x1="8.89" y1="-9.042" x2="6.35" y2="-9.042" width="0" layer="19" extent="1-1"/>
 <wire x1="12.7" y1="-9.042" x2="8.89" y2="-9.042" width="0" layer="19" extent="1-1"/>
@@
 <wire x1="22.22" y1="-3.81" x2="22.86" y2="-6.62" width="0" layer="19" extent="1-1"/>
 </signal>
-<signal name="N$8">
-<contactref element="R8" pad="1"/>
-<contactref element="R10" pad="1"/>
-<contactref element="R9" pad="1"/>
-<contactref element="R11" pad="1"/>
-<contactref element="T2" pad="7"/>
-<contactref element="C7" pad="2"/>
-<wire x1="-8.89" y1="-7.468" x2="-48.13" y2="-43.18" width="0" layer="19" extent="1-1"/>
-<wire x1="-8.738" y1="-5.08" x2="-8.89" y2="-7.468" width="0" layer="19" extent="1-1"/>
-<wire x1="-6.35" y1="-7.468" x2="-8.89" y2="-7.468" width="0" layer="19" extent="1-1"/>
-<wire x1="-8.738" y1="-2.54" x2="-8.738" y2="-5.08" width="0" layer="19" extent="1-1"/>
-<wire x1="-2.6162" y1="-6.35" x2="-6.35" y2="-7.468" width="0" layer="19" extent="1-1"/>
-</signal>
 <signal name="N$9">
 <contactref element="R11" pad="2"/>
@@
 <contactref element="C6" pad="1"/>
 <contactref element="C8" pad="1"/>
-<wire x1="2.6162" y1="5.08" x2="-50.93" y2="-49.53" width="0" layer="19" extent="1-1"/>
+<contactref element="T2" pad="1"/>
+<wire x1="1.8542" y1="-2.921" x2="-50.93" y2="-49.53" width="0" layer="19" extent="1-1"/>
+<wire x1="2.6162" y1="5.08" x2="1.8542" y2="-2.921" width="0" layer="19" extent="1-1"/>
 <wire x1="8.21" y1="5.08" x2="2.6162" y2="5.08" width="0" layer="19" extent="1-1"/>
 </signal>
+<signal name="N$8">
+<contactref element="R1" pad="1"/>
+<contactref element="R3" pad="1"/>
+<contactref element="R2" pad="1"/>
+<contactref element="R4" pad="1"/>
+<contactref element="T2" pad="8"/>
+<contactref element="C8" pad="2"/>
+<wire x1="2.6162" y1="-6.35" x2="-48.13" y2="-49.53" width="0" layer="19" extent="1-1"/>
+<wire x1="6.35" y1="-6.198" x2="2.6162" y2="-6.35" width="0" layer="19" extent="1-1"/>
+<wire x1="8.89" y1="-6.198" x2="6.35" y2="-6.198" width="0" layer="19" extent="1-1"/>
+<wire x1="8.738" y1="-3.81" x2="8.89" y2="-6.198" width="0" layer="19" extent="1-1"/>
+<wire x1="8.738" y1="-1.27" x2="8.738" y2="-3.81" width="0" layer="19" extent="1-1"/>
+</signal>
 </signals>
