File: EAGLE CAD/Modular_RFPA_v106.sch (EAGLE design)
At the start: 197 parts, among them IC301 74AHC1G14DBV, IC302 LM324D, J401 FUSE_2P, J402 KK_PCFAN, Q101 IRF520N, Q102 IRF630, Q201 IRF630, Q202 IRF630, Q301 BSS123, T101 HP4_TRAFO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

Commit message: copy "R" variants to "R90"
Parts:
- R401: value (none) -> 1K; device resistor:R-US_0817/7V -> MDT_R:R90R-1.0K-1%-1206-0.25WR1206
- R402, R403, R404, R405: device MDT_R:RR-1.0K-1%-1206-0.25WR1206 -> MDT_R:R90R-1.0K-1%-1206-0.25WR1206
- R408: device MDT_R:RR-1.0K-0.1%-0805-0.1W0805_IPC -> MDT_R:R90R-1.0K-0.1%-0805-0.1W0805_IPC
Other:
- moved on the sheet: R402, R403, R404, R405, R408
Changed lines of the file:
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@@
 <part name="D401" library="diode" deviceset="SCHOTTKY-DIODE" device="SMC"/>
 <part name="SUPPLY402" library="supply2" deviceset="GND" device=""/>
-<part name="R401" library="resistor" deviceset="R-US_" device="0817/7V"/>
+<part name="R401" library="MDT_R" deviceset="R90" device="R1206" technology="R-1.0K-1%-1206-0.25W" value="1K"/>
 <part name="C401" library="rcl" deviceset="CPOL-US" device="E10-25" value="3300uF"/>
 <part name="SUPPLY403" library="supply2" deviceset="GND" device=""/>
@@
 <part name="C408" library="MDT_C" deviceset="C" device="C2220_CKG57N" technology="CC-10U-100V-20%-2220-X7T" value="10uF"/>
 <part name="SUPPLY412" library="supply2" deviceset="GND" device=""/>
-<part name="R402" library="MDT_R" deviceset="R" device="R1206" technology="R-1.0K-1%-1206-0.25W" value="1K"/>
-<part name="R403" library="MDT_R" deviceset="R" device="R1206" technology="R-1.0K-1%-1206-0.25W" value="1K"/>
+<part name="R402" library="MDT_R" deviceset="R90" device="R1206" technology="R-1.0K-1%-1206-0.25W" value="1K"/>
+<part name="R403" library="MDT_R" deviceset="R90" device="R1206" technology="R-1.0K-1%-1206-0.25W" value="1K"/>
 <part name="IC301" library="74xx-little-us" deviceset="74*1G14" device="DBV" technology="AHC"/>
 <part name="R120" library="MDT_R" deviceset="R" device="R2512" technology="R-1K-1%-2512-1W" value="1K">
@@
 <part name="P+404" library="supply1" deviceset="+12V" device=""/>
 <part name="P+403" library="supply1" deviceset="+5V" device=""/>
-<part name="R408" library="MDT_R" deviceset="R" device="0805_IPC" technology="R-1.0K-0.1%-0805-0.1W" value="1.0K"/>
+<part name="R408" library="MDT_R" deviceset="R90" device="0805_IPC" technology="R-1.0K-0.1%-0805-0.1W" value="1.0K"/>
 <part name="SUPPLY405" library="supply2" deviceset="GND" device=""/>
 <part name="SUPPLY406" library="supply2" deviceset="GND" device=""/>
@@
 <part name="SUPPLY314" library="supply2" deviceset="GND" device=""/>
 <part name="P+305" library="supply1" deviceset="+5V" device=""/>
-<part name="R405" library="MDT_R" deviceset="R" device="R1206" technology="R-1.0K-1%-1206-0.25W" value="1K"/>
+<part name="R405" library="MDT_R" deviceset="R90" device="R1206" technology="R-1.0K-1%-1206-0.25W" value="1K"/>
 <part name="C402" library="MDT_C" deviceset="C" device="C2220_CKG57N" technology="CC-10U-100V-20%-2220-X7T" value="10uF"/>
 <part name="SUPPLY404" library="supply2" deviceset="GND" device=""/>
@@
 </part>
 <part name="R304" library="MDT_R" deviceset="R" device="0805_IPC" technology="R-1.0K-0.1%-0805-0.1W" value="1.0K"/>
-<part name="R404" library="MDT_R" deviceset="R" device="R1206" technology="R-1.0K-1%-1206-0.25W" value="1K"/>
+<part name="R404" library="MDT_R" deviceset="R90" device="R1206" technology="R-1.0K-1%-1206-0.25W" value="1K"/>
 <part name="D402" library="diode" deviceset="GP15" device=""/>
 <part name="C404" library="MDT_C" deviceset="C" device="C1210" technology="CC-6.8U-50V-10%-1210-X7S" value="6.8uF"/>
@@
 <instance part="C408" gate="G$1" x="228.6" y="165.1"/>
 <instance part="SUPPLY412" gate="GND" x="228.6" y="157.48" smashed="yes"/>
-<instance part="R402" gate="G$1" x="172.72" y="137.16" rot="R90"/>
-<instance part="R403" gate="G$1" x="172.72" y="101.6" rot="R90"/>
+<instance part="R402" gate="G$1" x="172.72" y="137.16"/>
+<instance part="R403" gate="G$1" x="172.72" y="101.6"/>
 <instance part="X401" gate="-1" x="81.28" y="175.26"/>
 <instance part="X401" gate="-2" x="81.28" y="170.18"/>
@@
 <attribute name="VALUE" x="259.08" y="66.04" size="1.778" layer="96" align="top-center"/>
 </instance>
-<instance part="R408" gate="G$1" x="269.24" y="55.88" smashed="yes" rot="R90">
-<attribute name="NAME" x="269.24" y="61.341" size="1.6764" layer="95" align="bottom-center"/>
-<attribute name="VALUE" x="269.24" y="59.309" size="1.6764" layer="96" align="bottom-center"/>
-<attribute name="PACKAGE" x="269.24" y="57.277" size="1.6764" layer="97" align="bottom-center"/>
-<attribute name="BOM" x="273.812" y="57.15" size="1.6764" layer="97" rot="R90"/>
-<attribute name="TOL" x="271.78" y="57.15" size="1.6764" layer="97" rot="R90"/>
-</instance>
+<instance part="R408" gate="G$1" x="269.24" y="55.88"/>
 <instance part="SUPPLY405" gate="GND" x="185.42" y="124.46" smashed="yes"/>
 <instance part="SUPPLY406" gate="GND" x="185.42" y="88.9" smashed="yes"/>
@@
 <instance part="SUPPLY418" gate="GND" x="259.08" y="157.48" smashed="yes"/>
 <instance part="SUPPLY419" gate="GND" x="274.32" y="157.48" smashed="yes"/>
-<instance part="R405" gate="G$1" x="215.9" y="185.42" rot="R90"/>
+<instance part="R405" gate="G$1" x="215.9" y="185.42"/>
 <instance part="C402" gate="G$1" x="170.18" y="165.1" smashed="yes">
 <attribute name="NAME" x="172.72" y="168.402" size="1.6764" layer="95"/>
@@
 <instance part="SUPPLY416" gate="GND" x="241.3" y="78.74" smashed="yes"/>
 <instance part="SUPPLY415" gate="GND" x="241.3" y="114.3" smashed="yes"/>
-<instance part="R404" gate="G$1" x="215.9" y="195.58" rot="R90"/>
+<instance part="R404" gate="G$1" x="215.9" y="195.58"/>
 <instance part="D402" gate="1" x="157.48" y="149.86" rot="R90"/>
 <instance part="C404" gate="G$1" x="185.42" y="93.98" rot="MR0"/>

Commit message: More schematic/library changes
Parts:
- D401: value (none) -> D-SCHOTTKYSK810L-TPSMC; device diode:SCHOTTKY-DIODESMC -> MDT_Diode:D-SCHOTTKYSK810L-TPSMC
- D402: value GP15 -> D-ZENER1N5355B-TPDO15-12; device diode:GP15 -> MDT_Diode:D-ZENER1N5355B-TPDO15-12
- L401: device MDT_L:L -> MDT_L:LL-3.3U-FERRITE-20%-12.5X12.5MM-10.5A
- L402: device MDT_L:L -> MDT_L:LL-22U-FERRITE-20%-12.5X12.5MM-4A
- R401, R402, R403, R404: value 1K -> 1.0
- R405: value 1K -> 0.5
- R406: value 1.0K -> 2K
- R407: value 1.0K -> 590
- R408: value 1.0K -> 10K
Connections:
- net GND: now also D401.A1; no longer D401.A
- net N$28: now also D402.A1; no longer D402.A
- net N$44: now also D401.C1; no longer D401.C
- net N$46: now also D402.C1; no longer D402.C
Other:
- moved on the sheet: H401, H402, H403, H404, R404, R405

Commit message: .
Parts:
- R401: device MDT_R:R90R-1.0K-1%-1206-0.25WR1206 -> resistor:R-US_0817/7V
Changed lines of the file:
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@@
 <grid distance="0.1" unitdist="inch" unit="inch" style="lines" multiple="1" display="no" altdistance="0.01" altunitdist="inch" altunit="inch"/>
 <layers>
-<layer number="1" name="Top" color="4" fill="1" visible="yes" active="no"/>
-<layer number="2" name="Route2" color="1" fill="3" visible="yes" active="no"/>
-<layer number="3" name="Route3" color="4" fill="3" visible="yes" active="no"/>
-<layer number="4" name="Route4" color="1" fill="4" visible="yes" active="no"/>
-<layer number="5" name="Route5" color="4" fill="4" visible="yes" active="no"/>
-<layer number="6" name="Route6" color="1" fill="8" visible="yes" active="no"/>
-<layer number="7" name="Route7" color="4" fill="8" visible="yes" active="no"/>
-<layer number="8" name="Route8" color="1" fill="2" visible="yes" active="no"/>
-<layer number="9" name="Route9" color="4" fill="2" visible="yes" active="no"/>
-<layer number="10" name="Route10" color="1" fill="7" visible="yes" active="no"/>
-<layer number="11" name="Route11" color="4" fill="7" visible="yes" active="no"/>
-<layer number="12" name="Route12" color="1" fill="5" visible="yes" active="no"/>
-<layer number="13" name="Route13" color="4" fill="5" visible="yes" active="no"/>
-<layer number="14" name="Route14" color="1" fill="6" visible="yes" active="no"/>
-<layer number="15" name="Route15" color="4" fill="6" visible="yes" active="no"/>
-<layer number="16" name="Bottom" color="1" fill="1" visible="yes" active="no"/>
-<layer number="17" name="Pads" color="2" fill="1" visible="yes" active="no"/>
-<layer number="18" name="Vias" color="2" fill="1" visible="yes" active="no"/>
-<layer number="19" name="Unrouted" color="6" fill="1" visible="yes" active="no"/>
-<layer number="20" name="Dimension" color="15" fill="1" visible="yes" active="no"/>
-<layer number="21" name="tPlace" color="7" fill="1" visible="yes" active="no"/>
-<layer number="22" name="bPlace" color="7" fill="1" visible="yes" active="no"/>
-<layer number="23" name="tOrigins" color="15" fill="1" visible="yes" active="no"/>
-<layer number="24" name="bOrigins" color="15" fill="1" visible="yes" active="no"/>
-<layer number="25" name="tNames" color="7" fill="1" visible="yes" active="no"/>
-<layer number="26" name="bNames" color="7" fill="1" visible="yes" active="no"/>
-<layer number="27" name="tValues" color="7" fill="1" visible="yes" active="no"/>
-<layer number="28" name="bValues" color="7" fill="1" visible="yes" active="no"/>
+<layer number="1" name="Top" color="4" fill="1" visible="no" active="no"/>
+<layer number="2" name="Route2" color="1" fill="3" visible="no" active="no"/>
+<layer number="3" name="Route3" color="4" fill="3" visible="no" active="no"/>
+<layer number="4" name="Route4" color="1" fill="4" visible="no" active="no"/>
+<layer number="5" name="Route5" color="4" fill="4" visible="no" active="no"/>
+<layer number="6" name="Route6" color="1" fill="8" visible="no" active="no"/>
+<layer number="7" name="Route7" color="4" fill="8" visible="no" active="no"/>
+<layer number="8" name="Route8" color="1" fill="2" visible="no" active="no"/>
+<layer number="9" name="Route9" color="4" fill="2" visible="no" active="no"/>
+<layer number="10" name="Route10" color="1" fill="7" visible="no" active="no"/>
+<layer number="11" name="Route11" color="4" fill="7" visible="no" active="no"/>
+<layer number="12" name="Route12" color="1" fill="5" visible="no" active="no"/>
+<layer number="13" name="Route13" color="4" fill="5" visible="no" active="no"/>
+<layer number="14" name="Route14" color="1" fill="6" visible="no" active="no"/>
+<layer number="15" name="Route15" color="4" fill="6" visible="no" active="no"/>
+<layer number="16" name="Bottom" color="1" fill="1" visible="no" active="no"/>
+<layer number="17" name="Pads" color="2" fill="1" visible="no" active="no"/>
+<layer number="18" name="Vias" color="2" fill="1" visible="no" active="no"/>
+<layer number="19" name="Unrouted" color="6" fill="1" visible="no" active="no"/>
+<layer number="20" name="Dimension" color="15" fill="1" visible="no" active="no"/>
+<layer number="21" name="tPlace" color="7" fill="1" visible="no" active="no"/>
+<layer number="22" name="bPlace" color="7" fill="1" visible="no" active="no"/>
+<layer number="23" name="tOrigins" color="15" fill="1" visible="no" active="no"/>
+<layer number="24" name="bOrigins" color="15" fill="1" visible="no" active="no"/>
+<layer number="25" name="tNames" color="7" fill="1" visible="no" active="no"/>
+<layer number="26" name="bNames" color="7" fill="1" visible="no" active="no"/>
+<layer number="27" name="tValues" color="7" fill="1" visible="no" active="no"/>
+<layer number="28" name="bValues" color="7" fill="1" visible="no" active="no"/>
 <layer number="29" name="tStop" color="7" fill="3" visible="no" active="no"/>
 <layer number="30" name="bStop" color="7" fill="6" visible="no" active="no"/>
@@
 <layer number="35" name="tGlue" color="7" fill="4" visible="no" active="no"/>
 <layer number="36" name="bGlue" color="7" fill="5" visible="no" active="no"/>
-<layer number="37" name="tTest" color="7" fill="1" visible="yes" active="no"/>
-<layer number="38" name="bTest" color="7" fill="1" visible="yes" active="no"/>
+<layer number="37" name="tTest" color="7" fill="1" visible="no" active="no"/>
+<layer number="38" name="bTest" color="7" fill="1" visible="no" active="no"/>
 <layer number="39" name="tKeepout" color="4" fill="11" visible="no" active="no"/>
 <layer number="40" name="bKeepout" color="1" fill="11" visible="no" active="no"/>
@@
 <layer number="44" name="Drills" color="7" fill="1" visible="no" active="no"/>
 <layer number="45" name="Holes" color="7" fill="1" visible="no" active="no"/>
-<layer number="46" name="Milling" color="3" fill="1" visible="yes" active="no"/>
-<layer number="47" name="Measures" color="7" fill="1" visible="yes" active="no"/>
-<layer number="48" name="Document" color="7" fill="1" visible="yes" active="no"/>
-<layer number="49" name="Reference" color="7" fill="1" visible="yes" active="no"/>
-<layer number="50" name="dxf" color="7" fill="1" visible="yes" active="no"/>
-<layer number="51" name="tDocu" color="7" fill="1" visible="yes" active="no"/>
-<layer number="52" name="bDocu" color="7" fill="1" visible="yes" active="no"/>
-<layer number="56" name="wert" color="7" fill="1" visible="yes" active="no"/>
+<layer number="46" name="Milling" color="3" fill="1" visible="no" active="no"/>
+<layer number="47" name="Measures" color="7" fill="1" visible="no" active="no"/>
+<layer number="48" name="Document" color="7" fill="1" visible="no" active="no"/>
+<layer number="49" name="Reference" color="7" fill="1" visible="no" active="no"/>
+<layer number="50" name="dxf" color="7" fill="1" visible="no" active="no"/>
+<layer number="51" name="tDocu" color="7" fill="1" visible="no" active="no"/>
+<layer number="52" name="bDocu" color="7" fill="1" visible="no" active="no"/>
+<layer number="56" name="wert" color="7" fill="1" visible="no" active="no"/>
 <layer number="90" name="Modules" color="5" fill="1" visible="yes" active="yes"/>
 <layer number="91" name="Nets" color="2" fill="1" visible="yes" active="yes"/>
@@
 </attributes>
 <variantdefs>
-<variantdef name="IRF520N_20W" current="yes"/>
+<variantdef name="IRF520N_20W"/>
 <variantdef name="IRF630_200W"/>
 </variantdefs>
@@
 <part name="D401" library="MDT_Diode" deviceset="D-SCHOTTKY" device="SMC" technology="SK810L-TP" value="D-SCHOTTKYSK810L-TPSMC"/>
 <part name="SUPPLY402" library="supply2" deviceset="GND" device=""/>
-<part name="R401" library="MDT_R" deviceset="R90" device="R1206" technology="R-1.0K-1%-1206-0.25W" value="1.0"/>
+<part name="R401" library="resistor" deviceset="R-US_" device="0817/7V" value="1.0"/>
 <part name="C401" library="rcl" deviceset="CPOL-US" device="E10-25" value="3300uF"/>
 <part name="SUPPLY403" library="supply2" deviceset="GND" device=""/>
