File: EAGLE CAD/Easy DICO/DICO_giangrandi_flipped_v100.brd (EAGLE design)
At the start: 50.8 x 44.5 mm, 32 parts, among them T1 TRAFO_CURRENTSENSEPA1005_NOCE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, T2 TRAFO_CURRENTSENSEPA1005_NOCE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

Commit message: dico and detector work
Parts:
- added X1, X2: 22-23-2021, con-molex:22-23-2021
- J1, J2, J3, J4: value (none) -> COAXSMA_0.375WIDE; device MDT_CON:BNC_EDGE -> MDT_CON:SMA_EDGE_0.375WIDE
- moved J2 6.35 mm to (-14.0, -22.9)
- moved J4 6.35 mm to (14.0, -22.9)
- moved J1 2.54 mm to (-25.4, 11.4)
- moved J3 2.54 mm to (25.4, 11.4)
Connections:
- net GND: now also J1.S1, J1.S2, J1.S3, J1.S4, J2.S1, J2.S2, J2.S3, J2.S4, J3.S1, J3.S2, J3.S3, J3.S4, J4.S1, J4.S2, J4.S3, J4.S4, X1.2, X2.2; no longer J1.G1, J1.G2, J1.G3, J1.G4, J2.G1, J2.G2, J2.G3, J2.G4, J3.G1, J3.G2, J3.G3, J3.G4, J4.G1, J4.G2, J4.G3, J4.G4
- net N$11: now also X1.1
- net N$7: now also X2.1
Routing:
- net N$7: track 15.9 -> 33.1 mm
- net N$11: track 15.8 -> 28.7 mm
Other:
- board size 50.8 x 44.5 mm -> 50.8 x 48.3 mm
