File: EAGLE CAD/Easy DICO/DICO_giangrandi_flipped_v100.sch (EAGLE design)
At the start: 32 parts, among them T1 TRAFO_CURRENTSENSEPA1005_NOCE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, T2 TRAFO_CURRENTSENSEPA1005_NOCE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

Commit message: dico and detector work
Parts:
- added X1, X2: 22-23-2021, con-molex:22-23-2021
- J1, J2, J3, J4: value (none) -> COAXSMA_0.375WIDE; device MDT_CON:COAXBNC_EDGE -> MDT_CON:COAXSMA_0.375WIDE
Connections:
- net GND: now also X1-2.S, X2-2.S
- net N$11: now also X1-1.S
- net N$7: now also X2-1.S
Other:
- moved on the sheet: C1, C2, D1, D2, R1, R16, R2, R3, R4, R5, R6, R7
