File: EAGLE CAD/Easy RFPA RevB/Modular_RFPA_RevB.brd (EAGLE design)
At the start: 152.4 x 152.4 mm, 189 parts, among them IC201 74AHC1G14DBV, IC202 LM324D, J1 FUSE_2P, J2 KK_PCFAN, Q1 IRF540, Q101 IRF540, Q102 IRF540, Q2 IRF540, Q201 BSS123, T1 HP4_TRAFO, T2 HP4_TRAFO, X101 HEATSINK_OMNI_DUAL30-75-D

Commit message: Resort eagle folder
Divide RFPA into revA and revB folders
Delete other versions
Parts:
- removed C1, C7: 22nF, MDT_C:C1206
- removed C12, C3, C9: 0.1uF, MDT_C:0805_IPC-7351B
- removed C13, C14, C15, C16: 47nF, MDT_C:C1206
- removed C18: 0.1uF, MDT_C:C1812
- removed D1: (no value), diode:DO41Z10
- removed D301: (no value), diode:SMC
- removed IC201: 74AHC1G14DBV, 74xx-little-us:SOT23-5
- removed IC202: LM324D, linear:SO14
- removed J2: KK_PCFAN, MDT_CON:47053-1000
- removed L4: 3.3uH, inductors:DR127
- removed L5: 22uH, inductors:DR127
- removed L6, L7: DR127, inductors:DR127
- removed LED1, LED2: (no value), led:LED5MM
- removed Q1: IRF540, transistor-power:TO220BV
- removed R10, R12, R22, R25, R27, R28, R29, R31, R8, R9: 1.0K, MDT_R:0805_IPC-7351B
- removed R13, R18, R19, R26, R5, R6: 1K, MDT_R:R1206
- removed R14, R15, R16, R2, R20, R3, R32, R36, R37, R38, R39, R7: 1K, MDT_R:R2512
- added C108, C115, C302, C305: 0.1uF, MDT_C:0805_IPC-7351B
- added C118, C119, C120: 0.1uF, MDT_C:C1812
- added C401: 3300uF, rcl:EB25D
- added C403, C404: 6.8uF, MDT_C:C1210
- added C405, C408: 10uF, MDT_C:C2220_CKG57N
- added C406, C407: 47nF, MDT_C:C1206
- added C409, C410: 22uF, rcl:E2,5-7
- added D401: D-SCHOTTKYSK810L-TPSMC, MDT_Diode:DO-214AB(SMC)
- added D402: D-ZENER1N5355B-TPDO15-12, MDT_Diode:DO15-12
- added IC401, IC402: (no value), v-reg:78XXS
- added J402: KK_PCFAN, MDT_CON:47053-1000
- added L103, L104: (no value), MDT_L:DR127
- added L401: 3.3uH, MDT_L:DR127
- added L402: 22uH, MDT_L:DR127
- added LED401, LED402: (no value), led:LED5MM
- added Q301: BSS123, transistor-small-signal:SOT23
- added R130, R131, R304, R305, R306, R307, R308, R310, R311, R312, R313, R314, R315, R316, R317: 1.0K, MDT_R:0805_IPC-7351B
- added R221, R222, R223, R224, R225, R226, R227, R228: 1K, MDT_R:R2512
- added R401: 1.0, resistor:P0817V
- added R402, R403, R404: 1.0, MDT_R:R1206
- added R406: 2K, MDT_R:0805_IPC-7351B
- added R407: 590, MDT_R:0805_IPC-7351B
- added R408: 10K, MDT_R:0805_IPC-7351B
- C111: value 22nF -> 0.1uF; device MDT_C:C1206 -> MDT_C:0805_IPC-7351B
- C113, C209, C210: value 0.1uF -> 22nF; device MDT_C:0805_IPC-7351B -> MDT_C:C1206
- C117: value 2.2uF -> 0.1uF; device MDT_C:C2220_CKG57N -> MDT_C:C1812
- C301: value 3300uF -> 0.1uF; device rcl:EB25D -> MDT_C:0805_IPC-7351B
- C303, C304: value 10uF -> 0.1uF; device MDT_C:C2220_CKG57N -> MDT_C:0805_IPC-7351B
- IC301: value (none) -> 74AHC1G14DBV; device v-reg:78XXS -> 74xx-little-us:SOT23-5
- IC302: value (none) -> LM324D; device v-reg:78XXS -> linear:SO14
- Q101: value IRF540 -> IRF520N
- Q102, Q202: value IRF540 -> IRF630
- Q201: value BSS123 -> IRF630; device transistor-small-signal:SOT23 -> transistor-power:TO220BV
- R101, R108, R110, R302, R303: value 1K -> 1.0K; device MDT_R:R1206 -> MDT_R:0805_IPC-7351B
- R107, R109, R111, R202, R203, R204, R205, R206: value 1.0K -> 1K; device MDT_R:0805_IPC-7351B -> MDT_R:R1206
- R117: value 1K -> 1.0K; device MDT_R:R2512 -> MDT_R:0805_IPC-7351B
- R125, R126, R217, R218, R219: value 1.0K -> 1K; device MDT_R:0805_IPC-7351B -> MDT_R:R2512
- R201: value (none) -> 1K; device rcl:RTRIM3299W -> MDT_R:R1206
- R301: value (none) -> 10K; device resistor:P0817V -> rcl:RTRIM3299W
- R405: value 0.33 -> 0.5
- moved R201 113.6 mm to (19.3, 55.6), turned to 270 degrees
- moved C304 113.0 mm to (110.7, 29.5), flipped to the top, turned to 180 degrees
- moved R203 96.7 mm to (20.8, 59.7), turned to 0 degrees
- moved C102 96.1 mm to (47.0, 10.2), turned to 270 degrees
- moved C201 90.9 mm to (25.9, 50.5), turned to 180 degrees
- moved C303 89.8 mm to (101.1, 33.0), turned to 90 degrees
- moved R205 88.7 mm to (22.4, 55.6), turned to 270 degrees
- moved R217 86.7 mm to (36.1, 64.8), turned to 0 degrees
- moved R218 86.4 mm to (36.1, 69.3), turned to 0 degrees
- moved C103 86.2 mm to (50.8, 10.2), turned to 270 degrees
- moved C209 77.7 mm to (43.2, 67.8), turned to 270 degrees
- moved R207 76.6 mm to (26.9, 47.0)
- moved R211 74.3 mm to (30.0, 58.7)
- moved R302 72.5 mm to (102.6, 13.2), turned to 90 degrees
- moved R101 71.8 mm to (50.8, 32.3), flipped to the bottom
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- renumbered C10 to C205, C11 to C202, C17 to C116, C19 to C411, C2 to C212, C20 to C412, C21 to C413, C22 to C306, C23 to C402, C4 to C206, C5 to C204, C6 to C203, C8 to C211, H1 to H401, H2 to H402, H3 to H403, H4 to H404, J1 to J401, J201 to J301, J202 to J302, JP201 to JP301, JP202 to JP302, L1 to L202, L2 to L201, LED3 to LED301, Q2 to Q202, R1 to R220, R11 to R230, R17 to R208, R21 to R213, R23 to R215, R24 to R229, R30 to R132, R33 to R128, R34 to R127, R35 to R129, R4 to R210, R40 to R405, R41 to R309, T1 to T101, T2 to T102, T201 to T301, T202 to T302, X1 to X401, X101 to X402
Connections:
- new net N$53: J302.C, R304.1
- net +12V: now also C305.1, C406.1, C409.+, IC302.4, IC401.OUT, J402.2, LED401.A; no longer C15.1, C210.1, IC202.4, IC301.OUT, J2.2, LED2.A
- net +5V: now also C407.1, C410.+, IC301.5, IC402.OUT, LED402.A, R301.3, R408.1; no longer C16.1, IC201.5, IC302.OUT, LED1.A, R201.3, R29.1
- net ABN1: now also R105.1, R202.1, R204.1; no longer R101.1, R13.1, R6.1
- net ABP1: now also R201.1, R203.1; no longer R19.1, R26.1
- net AN2: now also C107.2, R105.2, R107.1; no longer C103.2, R103.2, R105.1
- net AN3: now also C107.1, L102.1, R111.2, R115.1; no longer C103.1, L101.1, R108.2, R111.1
- net AN4: now also L102.2, Q102.G, R115.2, R120.1, R121.1; no longer L101.2, Q101.G, R113.2, R115.1, R118.1
- net AN5: now also Q102.S, R131.1; no longer Q101.S, R121.1
- net AN6: now also C115.1, R131.2; no longer C113.1, R125.2
- net AP3: now also L101.1, R109.2; no longer L102.1, R110.2
- net AP4: now also L101.2, Q101.G, R118.1; no longer L102.2, Q102.G, R120.1
- net AP5: now also Q101.S, R130.1; no longer Q102.S, R32.1
- net AP6: now also R130.2; no longer R126.2
- net BN2: now also R204.2, R206.1; no longer R5.1, R6.2
- net BN3: now also R212.1, R214.1; no longer R8.1, R9.1
- net BN4: now also R214.2, R216.1, R219.1; no longer R10.1, R7.1, R8.2
- net BN5: now also R222.1, R224.1, R226.1, R228.1; no longer R2.1, R3.1, R36.1, R37.1
- net BP2: now also R203.2, R205.1; no longer R18.1, R19.2
- net BP3: now also R211.1; no longer R22.1
- net BP4: now also Q201.G, R217.1, R218.1; no longer Q1.G, R14.1, R20.1
- net BP5: now also Q201.S, R221.1, R223.1, R225.1, R227.1; no longer Q1.S, R15.1, R16.1, R38.1, R39.1
- net DRAINS_NEG: now also C113.2, C117.2, C210.2, L104.1, Q102.D; no longer C1.2, C111.2, C18.2, L7.1, Q101.D
- net DRAINS_POS: now also C209.2, L103.1, Q101.D, Q201.D; no longer C7.2, L6.1, Q1.D, Q102.D
- net GBIAS: now also R108.1, R110.1, R207.1, R209.1, R316.2, R317.2; no longer R107.1, R109.1, R12.1, R218.2, R219.2, R25.1
- net GND: now also C108.2, C111.2, C115.2, C301.2, C302.2, C305.2, C401.-, C403.2, C404.2, C405.2, C406.2, C407.2, C408.2, C409.-, C410.-, D401.A, IC301.3, IC302.11, IC401.GND, IC402.GND, J402.1, Q301.2, R103.2, R107.2, R125.2, R126.2, R201.2, R202.2, R205.2, R206.2, R221.2, R222.2, R223.2, R224.2, R225.2, R226.2, R227.2, R228.2, R301.1, R307.2, R311.2, R312.1, R406.2, R407.2; no longer C102.2, C107.2, C113.2, C12.2, C13.2, C14.2, C15.2, C16.2, C210.2, C3.2, C301.-, C304.2, C9.2, D301.A, IC201.3, IC202.11, IC301.GND, IC302.GND, J2.1, Q201.2, R105.2, R121.2, R13.2, R15.2, R16.2, R18.2, R2.2, R201.1, R204.2, R211.2, R212.1, R26.2, R27.2, R28.2, R3.2, R31.2, R32.2, R36.2, R37.2, R38.2, R39.2, R5.2
- net N$1: now also IC302.1, R314.1, R315.1; no longer IC202.1, R216.1, R217.1
- net N$10: now also C108.1; no longer C107.1
- net N$12: now also R118.2; no longer R120.2
- net N$13: now also C106.1, R110.2, R111.1; no longer C102.1, R107.2, R108.1
- net N$14: now also C304.2, IC302.2, R312.2, R313.2, R317.1; no longer C209.2, IC202.2, R212.2, R214.2, R219.1
- net N$15: now also C303.1, IC302.3, R310.2, R311.1; no longer C208.1, IC202.3, R209.2, R211.1
- net N$16: now also IC302.10, R303.2, R306.1; no longer IC202.10, R203.2, R206.1
- net N$17: now also C111.1, R117.2; no longer C109.1, R115.2
- net N$18: now also IC302.8, R305.2, R308.1; no longer IC202.8, R205.2, R207.1
- net N$19: now also IC302.9, R302.2, R305.1; no longer IC202.9, R202.2, R205.1
- net N$2: now also R315.2, R316.1; no longer R217.2, R218.1
- net N$20: now also R302.1; no longer R202.1
- net N$21: now also R303.1; no longer R203.1
- net N$23: now also IC302.5, Q301.3, R308.2; no longer IC202.5, Q201.3, R207.2
- net N$24: now also IC301.4, Q301.1; no longer IC201.4, Q201.1
- net N$25: now also C301.1, IC302.12, R301.2; no longer C201.1, IC202.12, R201.2
- net N$26: now also IC302.13, IC302.14, R306.2; no longer IC202.13, IC202.14, R206.2
- net N$27: now also R101.1; no longer R31.1
- net N$28: now also D402.A, R402.1, R403.1; no longer D1.A, R302.1, R303.1
- net N$29: now also C119.1
- net N$3: now also IC301.2, R304.2, R307.1; no longer IC201.2, J302.C, R204.1
- net N$30: now also C120.1; no longer C117.1
- net N$31: now also C118.2, C119.2, C120.2; no longer C117.2
- net N$32: now also LED401.K, R406.1; no longer LED2.K, R27.1
- net N$33: now also LED402.K, R407.1; no longer LED1.K, R28.1
- net N$34: now also C101.2, C102.2, C103.2; no longer C101.1
- net N$35: now also R209.2; no longer R12.2
- net N$36: now also R212.2; no longer R9.2
- net N$38: now also C208.1, R216.2; no longer C3.1, R10.2
- net N$39: now also C210.1, R219.2; no longer C1.1, R7.2
- net N$4: now also C113.1, R120.2, R121.2; no longer C111.1, R117.2, R118.2
- net N$40: now also C201.1, R207.2; no longer C12.1, R25.2
- net N$41: now also C103.1; no longer C101.2
- net N$42: now also R211.2; no longer R22.2
- net N$43: now also C403.1, IC401.IN, R402.2; no longer C13.1, IC301.IN, R302.2
- net N$44: now also D401.K, R401.1; no longer D301.C, R301.1
- net N$46: now also C401.+, D402.C, L401.1, R401.2; no longer C301.+, D1.C, L4.1, R301.2
- net N$47: now also C405.1, L401.2, L402.1, R404.1; no longer C303.1, L4.2, L5.1
- net N$48: now also C207.1; no longer C9.1
- net N$49: now also C404.1, IC402.IN, R403.2; no longer C14.1, IC302.IN, R303.2
- net N$5: now also C109.1, R113.2; no longer C106.1, R111.2
- net N$50: now also C209.1, R217.2, R218.2; no longer C7.1, R14.2, R20.2
- net N$51: now also J402.3, R408.2; no longer J2.3, R29.2
- net N$52: now also C118.1
- net N$57: now also C101.1
- net N$6: now also IC302.6, IC302.7, R310.1; no longer IC202.6, IC202.7, R209.1
- net N$7: now also C304.1, R314.2; no longer C209.1, R216.2
- net N$8: now also R108.2, R109.1; no longer R109.2, R110.1
- net N$9: now also C302.1, R313.1; no longer C207.1, R214.1
- net VB: now also C117.1, C408.1, L103.2, L104.2, L402.2, R404.2; no longer C18.1, C304.1, L5.2, L6.2, L7.2
- net VB_CT1: now also C102.1
Routing:
- net N$57: track 23.4 -> 44.8 mm
- net VB_CT1: track 23.4 -> 44.2 mm
- net GND: track 91.7 -> 72.0 mm, vias 173 -> 177
- net N$52: track 23.4 -> 39.8 mm
- net N$29: track 23.4 -> 37.5 mm
- net +5V: track 146.4 -> 159.8 mm
- net N$31: track 12.3 -> 22.1 mm
- net N$34: track 5.10 -> 14.0 mm
- net +12V: track 136.0 -> 143.7 mm
- net N$3: track 15.0 -> 7.63 mm
- net N$28: track 22.7 -> 29.6 mm
- net N$53: track 0.00 -> 5.35 mm
- net N$51: track 15.3 -> 10.3 mm
- net N$47: track 26.6 -> 30.2 mm
- net N$30: track 9.07 -> 12.0 mm
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Other:
- board text added: "EASY RFPA FAB"
- board text removed: "DIY RFPA MODULE"
