File: EAGLE CAD/Easy RFPA RevB/Modular_RFPA_RevB.sch (EAGLE design)
At the start: 197 parts, among them IC201 74AHC1G14DBV, IC202 LM324D, J1 FUSE_2P, J2 KK_PCFAN, Q1 IRF630, Q101 IRF630, Q102 IRF520N, Q2 IRF630, Q201 BSS123, T1 HP4_TRAFO, T2 HP4_TRAFO, X101 HEATSINK_OMNI_DUAL30-75-D

Commit message: Resort eagle folder
Divide RFPA into revA and revB folders
Delete other versions
Parts:
- removed C1, C7: 22nF, MDT_C:CC-22N-250V-5%-1206-NP0C1206
- removed C12, C24, C25, C3, C9: 0.1uF, MDT_C:CC-0.1U-16V-0805-X7R0805_IPC
- removed D2: GP15, diode:GP15
- removed D301: (no value), diode:SCHOTTKY-DIODESMC
- removed H1, H2, H3, H4: MOUNT-PAD-SQUARE3.2, holes:MOUNT-PAD-SQUARE3.2
- removed IC201: 74AHC1G14DBV, 74xx-little-us:74AHC1G14DBV
- removed IC202: LM324D, linear:LM324D
- removed L4: 3.3uH, MDT_L:L
- removed L5: 22uH, MDT_L:L
- removed Q1: IRF630, transistor-power:IRF540
- removed R10, R12, R22, R25, R29, R31, R8, R9: 1.0K, MDT_R:RR-1.0K-0.1%-0805-0.1W0805_IPC
- removed R13, R18, R19, R26, R40, R43, R5, R6: 1K, MDT_R:RR-1.0K-1%-1206-0.25WR1206
- removed R14, R20, R32, R7: 1K, MDT_R:RR-1K-1%-2512-1WR2512
- added C108, C115, C302, C305: 0.1uF, MDT_C:CC-0.1U-16V-0805-X7R0805_IPC
- added C401: 3300uF, rcl:CPOL-USE10-25
- added C405, C408: 10uF, MDT_C:CCC-10U-100V-20%-2220-X7TC2220_CKG57N
- added D401: D-SCHOTTKYSK810L-TPSMC, MDT_Diode:D-SCHOTTKYSK810L-TPSMC
- added D402: D-ZENER1N5355B-TPDO15-12, MDT_Diode:D-ZENER1N5355B-TPDO15-12
- added H401, H402, H403, H404: MOUNT-PAD-SQUARE3.2, holes:MOUNT-PAD-SQUARE3.2
- added IC401, IC402: (no value), v-reg:78XXS
- added L401: 3.3uH, MDT_L:LL-3.3U-FERRITE-20%-12.5X12.5MM-10.5A
- added L402: 22uH, MDT_L:LL-22U-FERRITE-20%-12.5X12.5MM-4A
- added Q301: BSS123, transistor-small-signal:BSS123
- added R130, R131, R305, R306, R307, R308, R310, R311, R312, R313, R314, R315, R316, R317: 1.0K, MDT_R:RR-1.0K-0.1%-0805-0.1W0805_IPC
- added R401: 1.0, resistor:R-US_0817/7V
- added R402, R403, R404: 1.0, MDT_R:R90R-1.0K-1%-1206-0.25WR1206
- added R405: 0.5, MDT_R:R90R-1.0K-1%-1206-0.25WR1206
- added R408: 10K, MDT_R:R90R-1.0K-0.1%-0805-0.1W0805_IPC
- C106, C107, C201: BOM (none) -> INCLUDE
- C111: value 22nF -> 0.1uF; device MDT_C:CC-22N-250V-5%-1206-NP0C1206 -> MDT_C:CC-0.1U-16V-0805-X7R0805_IPC
- C113, C209, C210: value 0.1uF -> 22nF; device MDT_C:CC-0.1U-16V-0805-X7R0805_IPC -> MDT_C:CC-22N-250V-5%-1206-NP0C1206
- C207: BOM INCLUDE -> (none)
- C301: value 3300uF -> 0.1uF; device rcl:CPOL-USE10-25 -> MDT_C:CC-0.1U-16V-0805-X7R0805_IPC
- C303, C304: value 10uF -> 0.1uF; device MDT_C:CCC-10U-100V-20%-2220-X7TC2220_CKG57N -> MDT_C:CC-0.1U-16V-0805-X7R0805_IPC
- IC301: value (none) -> 74AHC1G14DBV; device v-reg:78XXS -> 74xx-little-us:74AHC1G14DBV
- IC302: value (none) -> LM324D; device v-reg:78XXS -> linear:LM324D
- Q101: value IRF630 -> IRF520N
- Q102: value IRF520N -> IRF630
- Q201: value BSS123 -> IRF630; device transistor-small-signal:BSS123 -> transistor-power:IRF540
- R101, R108, R110, R302, R303: value 1K -> 1.0K; device MDT_R:RR-1.0K-1%-1206-0.25WR1206 -> MDT_R:RR-1.0K-0.1%-0805-0.1W0805_IPC
- R107, R109, R111, R202, R203, R204, R205, R206: value 1.0K -> 1K; device MDT_R:RR-1.0K-0.1%-0805-0.1W0805_IPC -> MDT_R:RR-1.0K-1%-1206-0.25WR1206
- R117: value 1K -> 1.0K; device MDT_R:RR-1K-1%-2512-1WR2512 -> MDT_R:RR-1.0K-0.1%-0805-0.1W0805_IPC
- R125, R126, R217, R218, R219: value 1.0K -> 1K; device MDT_R:RR-1.0K-0.1%-0805-0.1W0805_IPC -> MDT_R:RR-1K-1%-2512-1WR2512
- R201: value 10K -> 1K; device rcl:R-TRIMM3299W -> MDT_R:RR-1.0K-1%-1206-0.25WR1206
- R301: value (none) -> 10K; device resistor:R-US_0817/7V -> rcl:R-TRIMM3299W
- R406: value 1.0K -> 2K
- R407: value 1.0K -> 590
- renumbered C10 to C205, C11 to C202, C13 to C403, C14 to C410, C15 to C406, C16 to C407, C17 to C116, C18 to C117, C19 to C411, C2 to C212, C20 to C412, C21 to C413, C22 to C306, C23 to C402, C26 to C120, C27 to C119, C28 to C101, C29 to C118, C30 to C404, C31 to C409, C4 to C206, C5 to C204, C6 to C203, C8 to C211, J1 to J401, J2 to J402, J201 to J301, J202 to J302, JP201 to JP301, JP202 to JP302, L1 to L202, L2 to L201, L6 to L103, L7 to L104, LED1 to LED402, LED2 to LED401, LED3 to LED301, Q2 to Q202, R1 to R220, R11 to R230, R15 to R223, R16 to R221, R17 to R208, R2 to R224, R21 to R213, R23 to R215, R24 to R229, R27 to R406, R28 to R407, R3 to R222, R30 to R132, R33 to R128, R34 to R127, R35 to R129, R36 to R226, R37 to R228, R38 to R225, R39 to R227, R4 to R210, R41 to R309, R42 to R304, T1 to T101, T2 to T102, T201 to T301, T202 to T302, X1 to X401, X101 to X402
Connections:
- net +12V: now also C305.1, IC302P.V+, IC401.OUT; no longer C210.1, IC202P.V+, IC301.OUT
- net +5V: now also IC301P.VCC, IC402.OUT, R301.E, R408.1; no longer IC201P.VCC, IC302.OUT, R201.E, R29.1
- net ABN1: now also R105.1, R202.1, R204.1; no longer R101.1, R13.1, R6.1
- net ABP1: now also R201.1, R203.1; no longer R19.1, R26.1
- net AN2: now also C107.2, R105.2, R107.1; no longer C103.2, R103.2, R105.1
- net AN3: now also C107.1, L102.1, R111.2, R115.1; no longer C103.1, L101.1, R108.2, R111.1
- net AN4: now also L102.2, Q102.G, R115.2, R120.1, R121.1; no longer L101.2, Q101.G, R113.2, R115.1, R118.1
- net AN5: now also Q102.S, R131.1; no longer Q101.S, R121.1
- net AN6: now also C115.1, R131.2; no longer C113.1, R125.2
- net AP3: now also L101.1, R109.2; no longer L102.1, R110.2
- net AP4: now also L101.2, Q101.G, R118.1; no longer L102.2, Q102.G, R120.1
- net AP5: now also Q101.S, R130.1; no longer Q102.S, R32.1
- net AP6: now also R130.2; no longer R126.2
- net BN2: now also R204.2, R206.1; no longer R5.1, R6.2
- net BN3: now also R212.1, R214.1; no longer R8.1, R9.1
- net BN4: now also R214.2, R216.1, R219.1; no longer R10.1, R7.1, R8.2
- net BP2: now also R203.2, R205.1; no longer R18.1, R19.2
- net BP3: now also R211.1; no longer R22.1
- net BP4: now also Q201.G, R217.1, R218.1; no longer Q1.G, R14.1, R20.1
- net BP5: now also Q201.S; no longer Q1.S
- net DRAINS_NEG: now also C113.2, C210.2, Q102.D; no longer C1.2, C111.2, Q101.D
- net DRAINS_POS: now also C209.2, Q101.D, Q201.D; no longer C7.2, Q1.D, Q102.D
- net GBIAS: now also R108.1, R110.1, R207.1, R209.1, R316.2, R317.2; no longer R107.1, R109.1, R12.1, R218.2, R219.2, R25.1
- net GND: now also C108.2, C111.2, C115.2, C301.2, C302.2, C305.2, C401.-, C405.2, C408.2, D401.A1, H401.MOUNT, H402.MOUNT, H403.MOUNT, H404.MOUNT, IC301P.GND, IC302P.V-, IC401.GND, IC402.GND, Q301.S, R103.2, R107.2, R125.2, R126.2, R201.2, R202.2, R205.2, R206.2, R301.A, R307.2, R311.2, R312.1; no longer C102.2, C107.2, C113.2, C12.2, C210.2, C3.2, C301.-, C304.2, C9.2, D301.A, H1.MOUNT, H2.MOUNT, H3.MOUNT, H4.MOUNT, IC201P.GND, IC202P.V-, IC301.GND, IC302.GND, Q201.S, R105.2, R121.2, R13.2, R18.2, R201.A, R204.2, R211.2, R212.1, R26.2, R31.2, R32.2, R5.2
- net N$1: now also IC302A.OUT, R314.1, R315.1; no longer IC202A.OUT, R216.1, R217.1
- net N$10: now also C108.1; no longer C107.1
- net N$12: now also R118.2; no longer R120.2
- net N$13: now also C106.1, R110.2, R111.1; no longer C102.1, R107.2, R108.1
- net N$14: now also C304.2, IC302A.-IN, R312.2, R313.2, R317.1; no longer C209.2, IC202A.-IN, R212.2, R214.2, R219.1
- net N$15: now also C303.1, IC302A.+IN, R310.2, R311.1; no longer C208.1, IC202A.+IN, R209.2, R211.1
- net N$16: now also IC302C.+IN, R303.2, R306.1; no longer IC202C.+IN, R203.2, R206.1
- net N$17: now also C111.1, R117.2; no longer C109.1, R115.2
- net N$18: now also IC302C.OUT, R305.2, R308.1; no longer IC202C.OUT, R205.2, R207.1
- net N$19: now also IC302C.-IN, R302.2, R305.1; no longer IC202C.-IN, R202.2, R205.1
- net N$2: now also R315.2, R316.1; no longer R217.2, R218.1
- net N$20: now also R302.1; no longer R202.1
- net N$21: now also R303.1; no longer R203.1
- net N$23: now also IC302B.+IN, Q301.D, R308.2; no longer IC202B.+IN, Q201.D, R207.2
- net N$24: now also IC301A.O, Q301.G; no longer IC201A.O, Q201.G
- net N$25: now also C301.1, IC302D.+IN, R301.S; no longer C201.1, IC202D.+IN, R201.S
- net N$26: now also IC302D.-IN, IC302D.OUT, R306.2; no longer IC202D.-IN, IC202D.OUT, R206.2
- net N$27: now also R101.1; no longer R31.1
- net N$28: now also D402.A1, R402.1, R403.1; no longer D2.A, R302.1, R303.1
- net N$3: now also IC301A.I, R307.1; no longer IC201A.I, R204.1
- net N$34: now also C102.2, C103.2; no longer C24.2, C25.2
- net N$35: now also R209.2; no longer R12.2
- net N$36: now also R212.2; no longer R9.2
- net N$38: now also C208.1, R216.2; no longer C3.1, R10.2
- net N$39: now also C210.1, R219.2; no longer C1.1, R7.2
- net N$4: now also C113.1, R120.2, R121.2; no longer C111.1, R117.2, R118.2
- net N$40: now also C201.1, R207.2; no longer C12.1, R25.2
- net N$41: now also C103.1; no longer C25.1
- net N$42: now also R211.2; no longer R22.2
- net N$43: now also IC401.IN, R402.2; no longer IC301.IN, R302.2
- net N$44: now also D401.C1, R401.1; no longer D301.C, R301.1
- net N$46: now also C401.+, D402.C1, L401.1, R401.2; no longer C301.+, D2.C, L4.1, R301.2
- net N$47: now also C405.1, L401.2, L402.1, R404.1, R405.1; no longer C303.1, L4.2, L5.1, R40.1, R43.1
- net N$48: now also C207.1; no longer C9.1
- net N$49: now also IC402.IN, R403.2; no longer IC302.IN, R303.2
- net N$5: now also C109.1, R113.2; no longer C106.1, R111.2
- net N$50: now also C209.1, R217.2, R218.2; no longer C7.1, R14.2, R20.2
- net N$51: now also R408.2; no longer R29.2
- net N$6: now also IC302B.-IN, IC302B.OUT, R310.1; no longer IC202B.-IN, IC202B.OUT, R209.1
- net N$7: now also C304.1, R314.2; no longer C209.1, R216.2
- net N$8: now also R108.2, R109.1; no longer R109.2, R110.1
- net N$9: now also C302.1, R313.1; no longer C207.1, R214.1
- net VB: now also C408.1, L402.2, R404.2, R405.2; no longer C304.1, L5.2, R40.2, R43.2
- net VB_CT1: now also C102.1; no longer C24.1
