File: EAGLE CAD/Easy RFPA RevA/Modular_RFPA_RevA.brd (EAGLE design)
At the start: 152.4 x 152.4 mm, 197 parts, among them IC301 74AHC1G14DBV, IC302 LM324D, J401 FUSE_2P, J402 KK_PCFAN, Q101 IRF520N, Q102 IRF630, Q201 IRF630, Q202 IRF630, Q301 BSS123, T101 HP4_TRAFO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

Commit message: adding more technologies...
Parts:
- removed T301, T302: (no value), transistor:SOT23-BEC
- added Q302: PNPSOT23_BEC, MDT_TRANS:SOT23R_INFINEON
- added Q303: NPNMMBT3904SOT23_BEC, MDT_TRANS:SOT23R_INFINEON
- L101, L102: value 1uH -> 47nH
- L103, L104: value (none) -> 3.3uH
- Q101, Q102, Q201, Q202: device transistor-power:TO220BV -> MDT_TRANS:TO220BV
- Q301: value BSS123 -> MOSFET_NBSS123SOT23; device transistor-small-signal:SOT23 -> MDT_TRANS:SOT23R_INFINEON
Connections:
- net +12V: now also Q303.3; no longer T301.C
- net GBIAS: now also Q302.2, Q303.2; no longer T301.E, T302.E
- net GND: now also Q302.3; no longer T302.C
- net N$2: now also Q302.1, Q303.1; no longer T301.B, T302.B

Commit message: more technologies....
Parts:
- removed IC302: LM324D, linear:SO14
- added U302: OPAMP_QUADTLV274IDSOIC14, MDT_IC:SO14
- IC401: value (none) -> LDO_3TERMMC78M12CTGTO220_VERT; device v-reg:78XXS -> MDT_IC:TO220BV
- IC402: value (none) -> LDO_3TERMMC78M05CTGTO220_VERT; device v-reg:78XXS -> MDT_IC:TO220BV
- LED301: value (none) -> LEDHLMP-3401-E0002T1_3/4; device led:LED5MM -> MDT_Diode:LED5MM
- LED401, LED402: value (none) -> LEDHLMP-3962-F0002T1_3/4; device led:LED5MM -> MDT_Diode:LED5MM
- renumbered IC301 to U301
Connections:
- net +12V: now also IC401.3, U302.4; no longer IC302.4, IC401.OUT
- net +5V: now also IC402.3; no longer IC402.OUT
- net GND: now also IC401.2, IC402.2, U302.11; no longer IC302.11, IC401.GND, IC402.GND
- net N$1: now also U302.1; no longer IC302.1
- net N$14: now also U302.2; no longer IC302.2
- net N$15: now also U302.3; no longer IC302.3
- net N$16: now also U302.10; no longer IC302.10
- net N$18: now also U302.8; no longer IC302.8
- net N$19: now also U302.9; no longer IC302.9
- net N$23: now also U302.5; no longer IC302.5
- net N$25: now also U302.12; no longer IC302.12
- net N$26: now also U302.13, U302.14; no longer IC302.13, IC302.14
- net N$43: now also IC401.1; no longer IC401.IN
- net N$49: now also IC402.1; no longer IC402.IN
- net N$6: now also U302.6, U302.7; no longer IC302.6, IC302.7

Commit message: .
Parts:
- C302, C303: value 0.1uF -> DNP
- C304: value 0.1uF -> 33pF
- C401: device rcl:EB25D -> MDT_C:EB25D
- C409, C410: device rcl:E2,5-7 -> MDT_C:E2,5-7
- R102, R103, R106, R107: value 1K -> 75; device MDT_R:R1206 -> MDT_R:1206_IPC-7351B
- R104, R105: value 1K -> 4.99; device MDT_R:R1206 -> MDT_R:1206_IPC-7351B
- R109, R111: value 1K -> 100; device MDT_R:R1206 -> MDT_R:1206_IPC-7351B
- R114, R115: value 1.0K -> 15
- R118: value 1K -> 2.74K
- R119: value 1K -> 270
- R401: device resistor:P0817V -> MDT_R:P0817V
- R402, R403, R404: value 1.0 -> 1K
- R405: value 0.5 -> 1K
- R406: value 2K -> 1.0K
- R407: value 590 -> 1.0K
- R408: value 10K -> 1.0K
- X402: value HEATSINK_OMNI_DUAL30-75-D -> HEATSINK_OMNI_DUALOMNI-UNI-30-75-D30-75-D

Commit message: .
Parts:
- C104, C106, C201, C203: value 0.1uF -> 22nF
- C105, C107, C202, C204: value 0.1uF -> 27nF
- C108, C109, C110, C111, C116, C117, C205, C206, C207, C208: value 0.1uF -> DNP
- C114, C115, C211, C212: value 0.1uF -> 10nF
- L201, L202: value 1uH -> 47nH
- R101, R132, R314: value 1.0K -> 0
- R108, R110, R207, R209, R316: value 1.0K -> 100
- R112, R113, R116, R117, R211, R215, R216: value 1.0K -> DNP
- R120, R217, R219: value 1K -> 2.74K
- R121, R218, R220: value 1K -> 270
- R122, R123, R124, R125, R126, R127, R221, R222, R223, R224, R225, R226: value 1K -> 2.7
- R128, R129, R227, R228: value 1K -> 3.3
- R201, R202, R205, R206: value 1K -> 75; device MDT_R:R1206 -> MDT_R:1206_IPC-7351B
- R203, R204: value 1K -> 4.99; device MDT_R:R1206 -> MDT_R:1206_IPC-7351B
- R208, R210: value 1K -> 100; device MDT_R:R1206 -> MDT_R:1206_IPC-7351B
- R213, R214: value 1.0K -> 15
- R312, R317: value 1.0K -> 10K
- R315: value 1.0K -> 10

Commit message: jellybean component values
Parts:
- C101, C102, C118, C119: value 0.1uF -> DNP
- C103, C120: value 0.1uF -> 3nF
- R302, R303, R305, R306: value 1.0K -> 10K
- R307: value 1.0K -> 100K
- R309: value 1.0K -> 150
- R311, R313: value 1.0K -> DNP
- R402, R403: value 1K -> 1.0
- R404: value 1K -> 1.0; device MDT_R:R1206 -> MDT_R:1206_IPC-7351B
- R405: value 1K -> 0.5; device MDT_R:R1206 -> MDT_R:1206_IPC-7351B
- R406: value 1.0K -> 2K
- R407: value 1.0K -> 590

Commit message: .
Parts:
- R130, R131: value 1.0K -> (none)
- R212: value 1.0K -> DNP
- R229, R230, R304, R308, R310: value 1.0K -> 1K
- R408: value 1.0K -> 10K
