File: EAGLE CAD/Easy RFPA RevA/Modular_RFPA_RevA.sch (EAGLE design)
At the start: 197 parts, among them IC301 74AHC1G14DBV, IC302 LM324D, J401 FUSE_2P, J402 KK_PCFAN, Q101 IRF520N, Q102 IRF630, Q201 IRF630, Q202 IRF630, Q301 BSS123, T101 HP4_TRAFO, T102 HP4_TRAFO, X402 HEATSINK_OMNI_DUAL30-75-D

Commit message: adding more technologies...
Parts:
- removed T301: (no value), transistor:BC808-NPN-SOT23-BEC
- removed T302: (no value), transistor:BC807-16-PNP-SOT23-BEC
- added Q302: PNPSOT23_BEC, MDT_TRANS:PNPSOT23_BEC
- added Q303: NPNMMBT3904SOT23_BEC, MDT_TRANS:NPNMMBT3904SOT23_BEC
- L101, L102: value 1uH -> 47nH; device MDT_L:L_CHIPL-1.0U-AIR-5%-1008-0.37A1008 -> MDT_L:L_CHIPL-47N-AIR-5%-1008-1A1008
- L103, L104: value (none) -> 3.3uH; device MDT_L:L -> MDT_L:LL-3.3U-FERRITE-20%-12.5X12.5MM-10.5A
- Q101, Q102, Q201, Q202: device transistor-power:IRF540 -> MDT_TRANS:MOSFET_NIRF630TO-220-VERT
- Q301: value BSS123 -> MOSFET_NBSS123SOT23; device transistor-small-signal:BSS123 -> MDT_TRANS:MOSFET_NBSS123SOT23
Connections:
- net +12V: now also Q303.C; no longer T301.C
- net GBIAS: now also Q302.E, Q303.E; no longer T301.E, T302.E
- net GND: now also Q302.C; no longer T302.C
- net N$2: now also Q302.B, Q303.B; no longer T301.B, T302.B

Commit message: more technologies....
Parts:
- removed IC302: LM324D, linear:LM324D
- added U302: OPAMP_QUADTLV274IDSOIC14, MDT_IC:OPAMP_QUADTLV274IDSOIC14
- IC401: value (none) -> LDO_3TERMMC78M12CTGTO220_VERT; device v-reg:78XXS -> MDT_IC:LDO_3TERMMC78M12CTGTO220_VERT
- IC402: value (none) -> LDO_3TERMMC78M05CTGTO220_VERT; device v-reg:78XXS -> MDT_IC:LDO_3TERMMC78M05CTGTO220_VERT
- LED301: value (none) -> LEDHLMP-3401-E0002T1_3/4; device led:LED5MM -> MDT_Diode:LEDHLMP-3401-E0002T1_3/4
- LED401, LED402: value (none) -> LEDHLMP-3962-F0002T1_3/4; device led:LED5MM -> MDT_Diode:LEDHLMP-3962-F0002T1_3/4
- renumbered IC301 to U301
Connections:
- net +12V: now also U302P.V+; no longer IC302P.V+
- net GND: now also U302P.V-; no longer IC302P.V-
- net N$1: now also U302A.OUT; no longer IC302A.OUT
- net N$14: now also U302A.-IN; no longer IC302A.-IN
- net N$15: now also U302A.+IN; no longer IC302A.+IN
- net N$16: now also U302C.+IN; no longer IC302C.+IN
- net N$18: now also U302C.OUT; no longer IC302C.OUT
- net N$19: now also U302C.-IN; no longer IC302C.-IN
- net N$23: now also U302B.+IN; no longer IC302B.+IN
- net N$25: now also U302D.+IN; no longer IC302D.+IN
- net N$26: now also U302D.-IN, U302D.OUT; no longer IC302D.-IN, IC302D.OUT
- net N$6: now also U302B.-IN, U302B.OUT; no longer IC302B.-IN, IC302B.OUT

Commit message: .
Parts:
- C302, C303: value 0.1uF -> DNP
- C304: value 0.1uF -> 33pF
- C401: device rcl:CPOL-USE10-25 -> MDT_C:CPOLC-3300U-63V-20%-25DX37L-ELECEB25D
- C409, C410: device rcl:CPOL-USE2.5-7 -> MDT_C:CPOLC-22U-63V-20%-6.3DX12.5L-ELECE2,5-7
- R102, R103, R106, R107: value 1K -> 75; device MDT_R:RR-1.0K-1%-1206-0.25WR1206 -> MDT_R:R1206_IPC
- R104, R105: value 1K -> 4.99; device MDT_R:RR-1.0K-1%-1206-0.25WR1206 -> MDT_R:R901206_IPC
- R109, R111: value 1K -> 100; device MDT_R:RR-1.0K-1%-1206-0.25WR1206 -> MDT_R:R1206_IPC
- R114: value 1.0K -> 15; device MDT_R:RR-1.0K-0.1%-0805-0.1W0805_IPC -> MDT_R:R900805_IPC
- R115: value 1.0K -> 15; device MDT_R:RR-1.0K-0.1%-0805-0.1W0805_IPC -> MDT_R:R90R-1.0K-0.1%-0805-0.1W0805_IPC
- R118: value 1K -> 2.74K; device MDT_R:RR-1K-1%-2512-1WR2512 -> MDT_R:R90R2512
- R119: value 1K -> 270; device MDT_R:RR-1K-1%-2512-1WR2512 -> MDT_R:R90R2512
- R120, R121: device MDT_R:RR-1K-1%-2512-1WR2512 -> MDT_R:R90R-1K-1%-2512-1WR2512
- R130: device MDT_R:RR-1.0K-0.1%-0805-0.1W0805_IPC -> MDT_R:R900805_IPC
- R131: device MDT_R:RR-1.0K-0.1%-0805-0.1W0805_IPC -> MDT_R:R90R-1.0K-0.1%-0805-0.1W0805_IPC
- R401: device resistor:R-US_0817/7V -> MDT_R:R90R-1.0-1%-AXIAL-3WP0817V
- R402, R403, R404: value 1.0 -> 1K
- R405: value 0.5 -> 1K
- R406: value 2K -> 1.0K
- R407: value 590 -> 1.0K
- R408: value 10K -> 1.0K
- X402: value HEATSINK_OMNI_DUAL30-75-D -> HEATSINK_OMNI_DUALOMNI-UNI-30-75-D30-75-D; device MDT_HEATSINK:HEATSINK_OMNI_DUAL30-75-D -> MDT_HEATSINK:HEATSINK_OMNI_DUALOMNI-UNI-30-75-D30-75-D
Other:
- note removed: "1N5355B-TP"
- note removed: "DR127-220-R"
- note removed: "DR127-3R3-R"
- note removed: "HLMP-3962-F0002‎"
- note removed: "LDOs"
- note removed: "PAC300001008FAC000"
- note removed: "SK810L-TP"
- moved on the sheet: C301, C302, C303, C304, C305, C306, J301, J302, JP301, JP302, LED301, Q301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

Commit message: .
Parts:
- C104, C106, C201, C203: value 0.1uF -> 22nF
- C105, C107, C202, C204: value 0.1uF -> 27nF
- C108, C109, C110, C111, C116, C117, C205, C206, C207, C208: value 0.1uF -> DNP
- C114, C115, C211, C212: value 0.1uF -> 10nF
- L201, L202: value 1uH -> 47nH; device MDT_L:L_CHIPL-1.0U-AIR-5%-1008-0.37A1008 -> MDT_L:L_CHIPL-47N-AIR-5%-1008-1A1008
- R101, R132, R314: value 1.0K -> 0
- R108, R110, R207, R209, R316: value 1.0K -> 100
- R112, R113, R116, R117, R211, R215, R216: value 1.0K -> DNP
- R120: value 1K -> 2.74K
- R121: value 1K -> 270
- R122, R123, R124, R125, R126, R127, R221, R222, R223, R224, R225, R226: value 1K -> 2.7
- R128, R129, R227, R228: value 1K -> 3.3
- R201, R202, R205, R206: value 1K -> 75; device MDT_R:RR-1.0K-1%-1206-0.25WR1206 -> MDT_R:R1206_IPC
- R203, R204: value 1K -> 4.99; device MDT_R:RR-1.0K-1%-1206-0.25WR1206 -> MDT_R:R901206_IPC
- R208, R210: value 1K -> 100; device MDT_R:RR-1.0K-1%-1206-0.25WR1206 -> MDT_R:R1206_IPC
- R213, R214: value 1.0K -> 15; device MDT_R:RR-1.0K-0.1%-0805-0.1W0805_IPC -> MDT_R:R90R-1.0K-0.1%-0805-0.1W0805_IPC
- R217, R219: value 1K -> 2.74K; device MDT_R:RR-1K-1%-2512-1WR2512 -> MDT_R:R90R-1K-1%-2512-1WR2512
- R218, R220: value 1K -> 270; device MDT_R:RR-1K-1%-2512-1WR2512 -> MDT_R:R90R-1K-1%-2512-1WR2512
- R229, R230: device MDT_R:RR-1.0K-0.1%-0805-0.1W0805_IPC -> MDT_R:R90R-1.0K-0.1%-0805-0.1W0805_IPC
- R312, R317: value 1.0K -> 10K
- R315: value 1.0K -> 10
Other:
- moved on the sheet: R203, R204, R213, R214, R217, R218, R219, R220, R229, R230

Commit message: jellybean component values
Parts:
- C101, C102, C118, C119: value 0.1uF -> DNP
- C103, C120: value 0.1uF -> 3nF
- R302, R303, R305, R306: value 1.0K -> 10K
- R307: value 1.0K -> 100K
- R309: value 1.0K -> 150
- R311, R313: value 1.0K -> DNP
- R402, R403: value 1K -> 1.0
- R404: value 1K -> 1.0; device MDT_R:R90R-1.0K-1%-1206-0.25WR1206 -> MDT_R:R901206_IPC
- R405: value 1K -> 0.5; device MDT_R:R90R-1.0K-1%-1206-0.25WR1206 -> MDT_R:R901206_IPC
- R406: value 1.0K -> 2K
- R407: value 1.0K -> 590
Other:
- note removed: "860010773010"
- note removed: "Values shown in this branch are for preamp uses one pair of IRF520N"
- note removed: "‎HLMP-3401-E0002‎"
- moved on the sheet: C301, C406, C407, C409, C410, J302, LED301, LED401, LED402, Q301, R301, R303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

Commit message: .
Parts:
- R101, R108, R110, R112, R113, R116, R117, R132, R207, R209, R211, R215, R216, R302, R303, R305, R306, R307, R309, R311, R312, R313, R314, R315, R316, R317, R406, R407: device MDT_R:RR-1.0K-0.1%-0805-0.1W0805_IPC -> MDT_R:RGEN0805_IPC
- R102, R103, R106, R107, R109, R111, R201, R202, R205, R206, R208, R210: device MDT_R:R1206_IPC -> MDT_R:RGEN1206_IPC
- R104, R105, R203, R204, R404, R405: device MDT_R:R901206_IPC -> MDT_R:R90GEN1206_IPC
- R114: device MDT_R:R900805_IPC -> MDT_R:R90GEN0805_IPC
- R115, R213, R214: device MDT_R:R90R-1.0K-0.1%-0805-0.1W0805_IPC -> MDT_R:R90GEN0805_IPC
- R118, R119: device MDT_R:R90R2512 -> MDT_R:R90GENR2512
- R120, R121, R217, R218, R219, R220: device MDT_R:R90R-1K-1%-2512-1WR2512 -> MDT_R:R90GENR2512
- R122, R123, R124, R125, R126, R127, R128, R129, R221, R222, R223, R224, R225, R226, R227, R228: device MDT_R:RR-1K-1%-2512-1WR2512 -> MDT_R:RGENR2512
- R130: value 1.0K -> (none); device MDT_R:R900805_IPC -> MDT_R:R90GEN0805_IPC
- R131: value 1.0K -> (none); device MDT_R:R90R-1.0K-0.1%-0805-0.1W0805_IPC -> MDT_R:R90GEN0805_IPC
- R212: value 1.0K -> DNP; device MDT_R:RR-1.0K-0.1%-0805-0.1W0805_IPC -> MDT_R:RGEN0805_IPC
- R229, R230: value 1.0K -> 1K; device MDT_R:R90R-1.0K-0.1%-0805-0.1W0805_IPC -> MDT_R:R90GEN0805_IPC
- R304, R308, R310: value 1.0K -> 1K; device MDT_R:RR-1.0K-0.1%-0805-0.1W0805_IPC -> MDT_R:RGEN0805_IPC
- R402, R403: device MDT_R:R90R-1.0K-1%-1206-0.25WR1206 -> MDT_R:R90GENR1206
- R408: value 1.0K -> 10K; device MDT_R:R90R-1.0K-0.1%-0805-0.1W0805_IPC -> MDT_R:R90GEN0805_IPC
