File: EAGLE CAD/Easy RFPA RevA S1/Easy_RFPA_RevA_S1.brd (EAGLE design)
At the start: 152.4 x 152.4 mm, 197 parts, among them J101 COAX112640BNC_EDGE, J102 COAX112640BNC_EDGE, J301 COAX112640BNC_EDGE, J302 COAX112640BNC_EDGE, J401 HDR_2X1282836-1282836-1, J402 KK_PCFAN, Q101 IRF520N, Q102 IRF630, Q201 IRF630, Q202 IRF630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

Commit message: S1 component values
Change component values for S1
Also fix a couple in S2
Export BOM and pdf for S1
Parts:
- C101, C118: value DNP -> 0.1uF
- C103, C120: value 3nF -> DNP
- C105, C107: value 27nF -> 12nF
- C112, C113: value 22nF -> 2.2nF
- C201, C203: value 22nF -> DNP
- C202, C204: value 27nF -> DNP
- C209, C210: value 2.2nF -> DNP
- C211, C212: value 10nF -> DNP
- L103, L104: value 3.3uH -> 22uH
- L201, L202: value 47nH -> DNP
- Q102: value IRF630 -> IRF520N
- R102, R103, R106, R107: value 75 -> 220
- R122, R123, R124, R125: value 2.7 -> 6.8
- R126, R127: value 2.7 -> 8.2
- R128, R129: value 3.3 -> 8.2
- R201, R202, R205, R206: value 75 -> DNP
- R203, R204: value 4.99 -> DNP
- R207, R208, R209, R210: value 100 -> DNP
- R213, R214: value 15 -> DNP
- R217, R219: value 2.74K -> DNP
- R218, R220: value 270 -> DNP
- R221, R222, R223, R224, R225, R226: value 2.7 -> DNP
- R227, R228: value 3.3 -> DNP
- R229, R230: value 1K -> DNP
