File: EAGLE CAD/Easy RFPA RevA S2/Easy_RFPA_RevA_S2.sch (EAGLE design)
At the start: 197 parts, among them J101 COAX112640BNC_EDGE, J102 COAX112640BNC_EDGE, J301 COAX112640BNC_EDGE, J302 COAX112640BNC_EDGE, J401 HDR_2X1282836-1282836-1, J402 KK_PCFAN, Q101 IRF520N, Q102 IRF630, Q201 IRF630, Q202 IRF630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

Commit message: S1 component values
Change component values for S1
Also fix a couple in S2
Export BOM and pdf for S1
Parts:
- C112, C113: value 22nF -> 2.2nF
- R118, R120, R217, R219: value 2.74K -> 330
Changed lines of the file:
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@@
 <part name="SUPPLY109" library="supply2" deviceset="GND" device=""/>
 <part name="SUPPLY107" library="supply2" deviceset="GND" device=""/>
-<part name="C113" library="MDT_C" deviceset="C" device="C1206" technology="GEN" value="22nF">
+<part name="C113" library="MDT_C" deviceset="C" device="C1206" technology="GEN" value="2.2nF">
 <attribute name="VOLTAGE" value="100V"/>
 </part>
@@
 <attribute name="VENDOR" value="Diodes Inc"/>
 </part>
-<part name="R120" library="MDT_R" deviceset="R90" device="R2512" technology="GEN" value="2.74K"/>
+<part name="R120" library="MDT_R" deviceset="R90" device="R2512" technology="GEN" value="330"/>
 <part name="R115" library="MDT_R" deviceset="R90" device="0805_IPC" technology="GEN" value="15"/>
 <part name="R113" library="MDT_R" deviceset="R" device="0805_IPC" technology="GEN" value="DNP">
@@
 <part name="SUPPLY108" library="supply2" deviceset="GND" device=""/>
 <part name="SUPPLY106" library="supply2" deviceset="GND" device=""/>
-<part name="C112" library="MDT_C" deviceset="C" device="C1206" technology="GEN" value="22nF">
+<part name="C112" library="MDT_C" deviceset="C" device="C1206" technology="GEN" value="2.2nF">
 <attribute name="VOLTAGE" value="100V"/>
 </part>
@@
 <part name="R106" library="MDT_R" deviceset="R" device="1206_IPC" technology="GEN" value="75"/>
 <part name="R104" library="MDT_R" deviceset="R90" device="1206_IPC" technology="GEN" value="4.99"/>
-<part name="R118" library="MDT_R" deviceset="R90" device="R2512" technology="GEN" value="2.74K"/>
+<part name="R118" library="MDT_R" deviceset="R90" device="R2512" technology="GEN" value="330"/>
 <part name="R114" library="MDT_R" deviceset="R90" device="0805_IPC" technology="GEN" value="15"/>
 <part name="R112" library="MDT_R" deviceset="R" device="0805_IPC" technology="GEN" value="DNP">
@@
 <variant name="IRF520N_20W" populate="no"/>
 </part>
-<part name="R219" library="MDT_R" deviceset="R90" device="R2512" technology="GEN" value="2.74K">
+<part name="R219" library="MDT_R" deviceset="R90" device="R2512" technology="GEN" value="330">
 <variant name="IRF520N_20W" populate="no"/>
 </part>
@@
 <variant name="IRF520N_20W" populate="no"/>
 </part>
-<part name="R217" library="MDT_R" deviceset="R90" device="R2512" technology="GEN" value="2.74K">
-<variant name="IRF520N_20W" populate="no"/>
-</part>
+<part name="R217" library="MDT_R" deviceset="R90" device="R2512" technology="GEN" value="330">
+<variant name="IRF520N_20W" populate="no"/>
+</part>
