File: EAGLE CAD/Easy RFPA RevB S2/Easy_RFPA_RevB_S2.sch (EAGLE design)
At the start: 197 parts, among them J101 COAX112640BNC_EDGE, J102 COAX112640BNC_EDGE, J301 COAX112640BNC_EDGE, J302 COAX112640BNC_EDGE, J401 HDR_2X1282836-1282836-1, J402 KK_PCFAN, Q101 IRF520N, Q102 IRF630, Q201 IRF630, Q202 IRF630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

Commit message: Work on revB
revB is basically the same as revA, except will have soldermask and silkscreen. Some components are moved around to make room for labels. Name labels updated in libraries.
Parts:
- TP10: value PROBE_TPTP_5MM -> PROBE_TPTP_7P5MM; device MDT_CON:PROBE_TPTP_5MM -> MDT_CON:PROBE_TPTP_7P5MM
- TP17: value PROBE_TPTP_7P5MM -> PROBE_TPTP_5MM; device MDT_CON:PROBE_TPTP_7P5MM -> MDT_CON:PROBE_TPTP_5MM
Changed lines of the file:
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@@
 <grid distance="0.1" unitdist="inch" unit="inch" style="lines" multiple="1" display="no" altdistance="0.01" altunitdist="inch" altunit="inch"/>
 <layers>
-<layer number="1" name="Top" color="4" fill="1" visible="no" active="no"/>
-<layer number="2" name="Route2" color="1" fill="3" visible="no" active="no"/>
-<layer number="3" name="Route3" color="4" fill="3" visible="no" active="no"/>
-<layer number="4" name="Route4" color="1" fill="4" visible="no" active="no"/>
-<layer number="5" name="Route5" color="4" fill="4" visible="no" active="no"/>
-<layer number="6" name="Route6" color="1" fill="8" visible="no" active="no"/>
-<layer number="7" name="Route7" color="4" fill="8" visible="no" active="no"/>
-<layer number="8" name="Route8" color="1" fill="2" visible="no" active="no"/>
-<layer number="9" name="Route9" color="4" fill="2" visible="no" active="no"/>
-<layer number="10" name="Route10" color="1" fill="7" visible="no" active="no"/>
-<layer number="11" name="Route11" color="4" fill="7" visible="no" active="no"/>
-<layer number="12" name="Route12" color="1" fill="5" visible="no" active="no"/>
-<layer number="13" name="Route13" color="4" fill="5" visible="no" active="no"/>
-<layer number="14" name="Route14" color="1" fill="6" visible="no" active="no"/>
-<layer number="15" name="Route15" color="4" fill="6" visible="no" active="no"/>
-<layer number="16" name="Bottom" color="1" fill="1" visible="no" active="no"/>
-<layer number="17" name="Pads" color="2" fill="1" visible="no" active="no"/>
-<layer number="18" name="Vias" color="2" fill="1" visible="no" active="no"/>
-<layer number="19" name="Unrouted" color="6" fill="1" visible="no" active="no"/>
-<layer number="20" name="Dimension" color="15" fill="1" visible="no" active="no"/>
-<layer number="21" name="tPlace" color="7" fill="1" visible="no" active="no"/>
-<layer number="22" name="bPlace" color="7" fill="1" visible="no" active="no"/>
-<layer number="23" name="tOrigins" color="15" fill="1" visible="no" active="no"/>
-<layer number="24" name="bOrigins" color="15" fill="1" visible="no" active="no"/>
-<layer number="25" name="tNames" color="7" fill="1" visible="no" active="no"/>
-<layer number="26" name="bNames" color="7" fill="1" visible="no" active="no"/>
-<layer number="27" name="tValues" color="7" fill="1" visible="no" active="no"/>
-<layer number="28" name="bValues" color="7" fill="1" visible="no" active="no"/>
+<layer number="1" name="Top" color="4" fill="1" visible="yes" active="no"/>
+<layer number="2" name="Route2" color="1" fill="3" visible="yes" active="no"/>
+<layer number="3" name="Route3" color="4" fill="3" visible="yes" active="no"/>
+<layer number="4" name="Route4" color="1" fill="4" visible="yes" active="no"/>
+<layer number="5" name="Route5" color="4" fill="4" visible="yes" active="no"/>
+<layer number="6" name="Route6" color="1" fill="8" visible="yes" active="no"/>
+<layer number="7" name="Route7" color="4" fill="8" visible="yes" active="no"/>
+<layer number="8" name="Route8" color="1" fill="2" visible="yes" active="no"/>
+<layer number="9" name="Route9" color="4" fill="2" visible="yes" active="no"/>
+<layer number="10" name="Route10" color="1" fill="7" visible="yes" active="no"/>
+<layer number="11" name="Route11" color="4" fill="7" visible="yes" active="no"/>
+<layer number="12" name="Route12" color="1" fill="5" visible="yes" active="no"/>
+<layer number="13" name="Route13" color="4" fill="5" visible="yes" active="no"/>
+<layer number="14" name="Route14" color="1" fill="6" visible="yes" active="no"/>
+<layer number="15" name="Route15" color="4" fill="6" visible="yes" active="no"/>
+<layer number="16" name="Bottom" color="1" fill="1" visible="yes" active="no"/>
+<layer number="17" name="Pads" color="2" fill="1" visible="yes" active="no"/>
+<layer number="18" name="Vias" color="2" fill="1" visible="yes" active="no"/>
+<layer number="19" name="Unrouted" color="6" fill="1" visible="yes" active="no"/>
+<layer number="20" name="Dimension" color="15" fill="1" visible="yes" active="no"/>
+<layer number="21" name="tPlace" color="7" fill="1" visible="yes" active="no"/>
+<layer number="22" name="bPlace" color="7" fill="1" visible="yes" active="no"/>
+<layer number="23" name="tOrigins" color="15" fill="1" visible="yes" active="no"/>
+<layer number="24" name="bOrigins" color="15" fill="1" visible="yes" active="no"/>
+<layer number="25" name="tNames" color="7" fill="1" visible="yes" active="no"/>
+<layer number="26" name="bNames" color="7" fill="1" visible="yes" active="no"/>
+<layer number="27" name="tValues" color="7" fill="1" visible="yes" active="no"/>
+<layer number="28" name="bValues" color="7" fill="1" visible="yes" active="no"/>
 <layer number="29" name="tStop" color="7" fill="3" visible="no" active="no"/>
 <layer number="30" name="bStop" color="7" fill="6" visible="no" active="no"/>
@@
 <layer number="35" name="tGlue" color="7" fill="4" visible="no" active="no"/>
 <layer number="36" name="bGlue" color="7" fill="5" visible="no" active="no"/>
-<layer number="37" name="tTest" color="7" fill="1" visible="no" active="no"/>
-<layer number="38" name="bTest" color="7" fill="1" visible="no" active="no"/>
+<layer number="37" name="tTest" color="7" fill="1" visible="yes" active="no"/>
+<layer number="38" name="bTest" color="7" fill="1" visible="yes" active="no"/>
 <layer number="39" name="tKeepout" color="4" fill="11" visible="no" active="no"/>
 <layer number="40" name="bKeepout" color="1" fill="11" visible="no" active="no"/>
@@
 <layer number="44" name="Drills" color="7" fill="1" visible="no" active="no"/>
 <layer number="45" name="Holes" color="7" fill="1" visible="no" active="no"/>
-<layer number="46" name="Milling" color="3" fill="1" visible="no" active="no"/>
-<layer number="47" name="Measures" color="7" fill="1" visible="no" active="no"/>
-<layer number="48" name="Document" color="7" fill="1" visible="no" active="no"/>
-<layer number="49" name="Reference" color="7" fill="1" visible="no" active="no"/>
-<layer number="50" name="dxf" color="7" fill="1" visible="no" active="no"/>
-<layer number="51" name="tDocu" color="7" fill="1" visible="no" active="no"/>
-<layer number="52" name="bDocu" color="7" fill="1" visible="no" active="no"/>
-<layer number="56" name="wert" color="7" fill="1" visible="no" active="no"/>
+<layer number="46" name="Milling" color="3" fill="1" visible="yes" active="no"/>
+<layer number="47" name="Measures" color="7" fill="1" visible="yes" active="no"/>
+<layer number="48" name="Document" color="7" fill="1" visible="yes" active="no"/>
+<layer number="49" name="Reference" color="7" fill="1" visible="yes" active="no"/>
+<layer number="50" name="dxf" color="7" fill="1" visible="yes" active="no"/>
+<layer number="51" name="tDocu" color="7" fill="1" visible="yes" active="no"/>
+<layer number="52" name="bDocu" color="7" fill="1" visible="yes" active="no"/>
+<layer number="56" name="wert" color="7" fill="1" visible="yes" active="no"/>
 <layer number="90" name="Modules" color="5" fill="1" visible="yes" active="yes"/>
 <layer number="91" name="Nets" color="2" fill="1" visible="yes" active="yes"/>
@@
 <part name="TP8" library="MDT_CON" deviceset="PROBE_TP" device="TP_7P5MM" value="PROBE_TPTP_7P5MM"/>
 <part name="TP9" library="MDT_CON" deviceset="PROBE_TP" device="TP_5MM"/>
-<part name="TP10" library="MDT_CON" deviceset="PROBE_TP" device="TP_5MM"/>
+<part name="TP10" library="MDT_CON" deviceset="PROBE_TP" device="TP_7P5MM" value="PROBE_TPTP_7P5MM"/>
 <part name="SUPPLY213" library="supply2" deviceset="GND" device=""/>
 <part name="SUPPLY214" library="supply2" deviceset="GND" device=""/>
@@
 <part name="TP16" library="MDT_CON" deviceset="PROBE_TP" device="TP_5MM"/>
 <part name="SUPPLY225" library="supply2" deviceset="GND" device=""/>
-<part name="TP17" library="MDT_CON" deviceset="PROBE_TP" device="TP_7P5MM" value="PROBE_TPTP_7P5MM"/>
+<part name="TP17" library="MDT_CON" deviceset="PROBE_TP" device="TP_5MM" value="PROBE_TPTP_5MM"/>
 <part name="SUPPLY226" library="supply2" deviceset="GND" device=""/>
 <part name="TP18" library="MDT_CON" deviceset="PROBE_TP" device="TP_5MM"/>

Commit message: Add thermal pads and heatsink clips to schematic
Also modify bom-ex old.ulp to not ignore parts which lack a package but have a part number
Other:
- note added: "Thermal pads and heatsink clips"
- moved on the sheet: X402
Changed lines of the file:
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@@
 </part>
 <part name="J401" library="MDT_CON" deviceset="HDR_2X1" device="282836-1" technology="282836-1"/>
+<part name="X1" library="MDT_HEATSINK" deviceset="THERMALPAD_TO220" device="" technology="DC0011/15-TI900-0.12-0"/>
+<part name="X2" library="MDT_HEATSINK" deviceset="THERMALPAD_TO220" device="" technology="DC0011/15-TI900-0.12-0"/>
+<part name="X3" library="MDT_HEATSINK" deviceset="THERMALPAD_TO220" device="" technology="DC0011/15-TI900-0.12-0"/>
+<part name="X4" library="MDT_HEATSINK" deviceset="THERMALPAD_TO220" device="" technology="DC0011/15-TI900-0.12-0"/>
+<part name="X5" library="MDT_HEATSINK" deviceset="HEATSINK_CLIP" device="" technology="OMNI-220C"/>
+<part name="X6" library="MDT_HEATSINK" deviceset="HEATSINK_CLIP" device="" technology="OMNI-220C"/>
+<part name="X7" library="MDT_HEATSINK" deviceset="HEATSINK_CLIP" device="" technology="OMNI-220C"/>
+<part name="X8" library="MDT_HEATSINK" deviceset="HEATSINK_CLIP" device="" technology="OMNI-220C"/>
 </parts>
 <sheets>
@@
 <plain>
 <text x="73.66" y="137.16" size="2.54" layer="94" align="center">Mounting holes</text>
-<text x="121.92" y="137.16" size="2.54" layer="94" align="center">Heatsink</text>
+<text x="375.92" y="180.34" size="2.54" layer="94" align="center">Heatsink</text>
 <text x="91.44" y="195.58" size="2.54" layer="94" align="center">Input protection
 Intended for 48VDC supply
@@
 Max duty cycle: 3.5% (500us, 70Hz rep rate, passive convection)
 Max pulse width: 1ms</text>
+<text x="375.92" y="139.7" size="2.54" layer="94" align="center">Thermal pads and heatsink clips</text>
 </plain>
 <instances>
@@
 <instance part="SUPPLY410" gate="GND" x="220.98" y="124.46" smashed="yes"/>
 <instance part="SUPPLY411" gate="GND" x="220.98" y="88.9" smashed="yes"/>
-<instance part="SUPPLY421" gate="GND" x="119.38" y="99.06" smashed="yes"/>
-<instance part="SUPPLY422" gate="GND" x="124.46" y="99.06" smashed="yes"/>
-<instance part="X402" gate="G$1" x="121.92" y="104.14"/>
+<instance part="SUPPLY421" gate="GND" x="373.38" y="147.32" smashed="yes"/>
+<instance part="SUPPLY422" gate="GND" x="378.46" y="147.32" smashed="yes"/>
+<instance part="X402" gate="G$1" x="375.92" y="152.4"/>
 <instance part="F401" gate="G$1" x="83.82" y="175.26" smashed="yes">
 <attribute name="NAME" x="83.82" y="180.34" size="1.778" layer="95" align="bottom-center"/>
@@
 <instance part="SUPPLY413" gate="GND" x="238.76" y="124.46" smashed="yes"/>
 <instance part="J401" gate="G$1" x="55.88" y="172.72" rot="MR0"/>
+<instance part="X1" gate="G$1" x="350.52" y="124.46"/>
+<instance part="X2" gate="G$1" x="350.52" y="101.6"/>
+<instance part="X3" gate="G$1" x="386.08" y="101.6"/>
+<instance part="X4" gate="G$1" x="386.08" y="124.46"/>
+<instance part="X5" gate="G$1" x="365.76" y="96.52"/>
+<instance part="X6" gate="G$1" x="365.76" y="119.38"/>
+<instance part="X7" gate="G$1" x="398.78" y="119.38"/>
+<instance part="X8" gate="G$1" x="398.78" y="96.52"/>
 </instances>
 <busses>

Commit message: Better docfield
I modified my docfield symbol (not included in the repo!)
I define a few global attributes:
BOMREV
FABREV
AUTHOR
DRAWING_NUMBER
Other:
- note added: "B"
Changed lines of the file:
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@@
 <schematic xreflabel="%F%N" xrefpart="/%S.%C%R">
 <attributes>
+<attribute name="AUTHOR" value="MDT"/>
+<attribute name="BOMREV" value="01"/>
+<attribute name="FABREV" value="B"/>
 </attributes>
 <variantdefs>
@@
 Max pulse width: 1ms</text>
 <text x="375.92" y="139.7" size="2.54" layer="94" align="center">Thermal pads and heatsink clips</text>
+<text x="414.02" y="7.62" size="2.54" layer="94">B</text>
 </plain>
 <instances>
